File: hw/buscom/buscom_mega32.sch (KiCad schematic (older format))
At the start: 19 parts, among them J201 JUMPER, J202 CONN_10X1, J203 CONN_10X1, J204 CONN_10X1, J205 CONN_8X1, J206 CONN_3X1, U201 ATMEGA324-TQFP44, U202 7,3728MHz

Commit message: changed tracknames.
Connections:
- net PB2 is gone; now on net HS: J205.4
- net CS: now also J205.5
- net GND: no longer J205.1
- net PB0: now also J205.1
- net PB1: now also J205.2; no longer J205.3
- net RESET: no longer J205.5
- net VCC: no longer J205.2
- net Reserve renamed TE
- net TE: now also J205.3
