File: hw/buscom-hub/buscom-hub.sch (KiCad schematic (older format))
At the start: 62 parts, among them J1 CONN-ISP-6, J10 CONN_1, J11 CONN_10X1, J2 JUMPER, J3 CONN_1, J4 CONN_1, J5 CONN_1, J6 CONN_1, J7 CONN_1, J8 CONN_1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

Commit message: aligned order of WAGO-connectors to comply with bus-connecting standard.
Parts:
- R1, R2, R24: value 1 -> 0
Connections:
- net labels added: +24V-1, +24V-2, 5V-1, 5V-2
- net labels removed: +24V(Master), +24V(Slave), +5V(Master), +5V(Slave)
Changed lines of the file:
@@
-EESchema Schematic File Version 2  date Di 14 Mai 2013 01:23:35 CEST
+EESchema Schematic File Version 2  date Fr 17 Mai 2013 23:21:25 CEST
 LIBS:connectors
 LIBS:ics_controller_atmel
@@
 Sheet 1 1
 Title ""
-Date "13 may 2013"
+Date "17 may 2013"
 Rev ""
 Comp ""
@@
 Comment4 ""
 $EndDescr
+Text Label 7100 1350 0    60   ~ 0
+5V-1
+Text Label 8100 1350 0    60   ~ 0
+5V-2
+Text Label 7050 750  0    60   ~ 0
++24V-1
+Text Label 8000 750  0    60   ~ 0
++24V-2
 Connection ~ 6750 6850
 Wire Wire Line
@@
 	0    1    1    0
 $EndComp
-Text Label 6850 1350 0    60   ~ 0
-+5V(Master)
-Text Label 8000 750  0    60   ~ 0
-+24V(Slave)
 Text Label 9800 6850 0    60   ~ 0
 GND2
-Text Label 6800 750  0    60   ~ 0
-+24V(Master)
 Text Notes 800  4350 0    60   ~ 0
 +24V(1)
@@
 Text Notes 10700 4350 0    60   ~ 0
 +24V(2)
-Text Label 8000 1350 0    60   ~ 0
-+5V(Slave)
 Text Label 4750 2250 0    60   ~ 0
 GND
@@
 P 7700 6850
 F 0 "R24" H 7650 6750 50  0000 L CNN
-F 1 "1" H 7675 6850 50  0000 L CNN
+F 1 "0" H 7675 6850 50  0000 L CNN
 F 2 "~" H 7825 6840 50  0001 L CNN
 F 3 "~" H 7825 6780 50  0001 L CNN
@@
 P 7700 750
 F 0 "R1" H 7650 650 50  0000 L CNN
-F 1 "1" H 7675 750 50  0000 L CNN
+F 1 "0" H 7675 750 50  0000 L CNN
 F 2 "~" H 7825 740 50  0001 L CNN
 F 3 "~" H 7825 680 50  0001 L CNN
@@
 P 7700 1350
 F 0 "R2" H 7650 1250 50  0000 L CNN
-F 1 "1" H 7675 1350 50  0000 L CNN
+F 1 "0" H 7675 1350 50  0000 L CNN
 F 2 "~" H 7825 1340 50  0001 L CNN
 F 3 "~" H 7825 1280 50  0001 L CNN
