File: hw/roomthermostat/businterface.sch (KiCad schematic (older format))
At the start: 17 parts, among them J301 CONN_1, J302 CONN_1, J303 CONN_1, J304 CONN_1, J305 JUMPER, U301 AM1S-2405, U302 MAX487

Commit message: updated businterface
Parts:
- removed D301: BRIDGE, symbol BRIDGE
- removed D302: P6SMB, symbol ZD
- renumbered R302 to R301, R301 to R302
Connections:
- wire segments 58 -> 51
Changed lines of the file:
@@
-EESchema Schematic File Version 2  date Sa 27 Apr 2013 15:07:17 CEST
-LIBS:connectors
-LIBS:display
-LIBS:encoder
-LIBS:ics_40xx
+EESchema Schematic File Version 2  date So 05 Mai 2013 15:34:25 CEST
 LIBS:ics_controller_atmel
 LIBS:ics_misc
-LIBS:ics_opamp
-LIBS:ics_opto
-LIBS:ics_peripheral
 LIBS:ics_regulator
 LIBS:power
-LIBS:relays
-LIBS:sensors
 LIBS:standard
-LIBS:transformer
-LIBS:transistors
-LIBS:roomthermostate-cache
-EELAYER 25  0
+LIBS:connectors
+LIBS:ics_peripheral
+LIBS:display
+LIBS:buscom-cache
+EELAYER 24  0
 EELAYER END
 $Descr A4 11700 8267
-encoding utf-8
-Sheet 3 2
+Sheet 3 3
 Title ""
-Date "27 apr 2013"
+Date "5 may 2013"
 Rev ""
 Comp ""
@@
 $EndDescr
 Wire Wire Line
-	2300 5125 2300 3350
-Wire Wire Line
-	2300 5475 2300 5600
+	3150 1350 3150 3600
+Connection ~ 3150 1450
+Wire Wire Line
+	2300 5150 2300 4300
+Wire Wire Line
+	3350 1850 3350 1750
+Wire Wire Line
+	3350 2850 3350 2750
+Wire Wire Line
+	2550 3350 2550 2750
+Wire Wire Line
+	1300 5950 1300 5050
+Wire Wire Line
+	3150 5850 3150 4700
+Connection ~ 3150 5100
+Wire Wire Line
+	3150 5100 2550 5100
+Wire Wire Line
+	2550 5100 2550 4950
+Wire Wire Line
+	4200 3800 4200 1450
+Wire Wire Line
+	4300 4500 4200 4500
+Wire Wire Line
+	4300 4300 3650 4300
+Wire Wire Line
+	3650 4000 4300 4000
+Connection ~ 1800 1900
+Wire Wire Line
+	2400 1900 1200 1900
+Wire Wire Line
+	2400 1900 2400 1650
+Wire Wire Line
+	2450 1450 2300 1450
+Wire Wire Line
+	2400 1650 2300 1650
+Wire Wire Line
+	1300 1450 1000 1450
+Connection ~ 1000 3900
+Wire Wire Line
+	1300 4550 1300 3900
+Wire Wire Line
+	1300 3900 1000 3900
+Connection ~ 3150 2750
+Connection ~ 2300 4300
+Wire Wire Line
+	740  4100 1100 4100
+Wire Wire Line
+	2100 4000 2100 4550
+Wire Wire Line
+	740  4000 1000 4000
+Connection ~ 2550 4300
+Wire Wire Line
+	2550 4550 2550 4300
+Wire Wire Line
+	2100 4950 2100 5600
+Connection ~ 2300 4300
+Wire Wire Line
+	2650 4000 1100 4000
+Wire Wire Line
+	2650 4300 1100 4300
+Connection ~ 2100 4000
+Wire Wire Line
+	1100 4300 1100 4200
+Wire Wire Line
+	740  4300 1000 4300
+Wire Wire Line
+	1100 4200 740  4200
+Wire Wire Line
+	2100 5600 2300 5600
+Wire Wire Line
+	2550 4000 2550 3750
+Connection ~ 2550 4000
+Wire Wire Line
+	1300 1650 1200 1650
+Wire Wire Line
+	1000 4000 1000 2550
+Wire Wire Line
+	3650 4100 3700 4100
+Wire Wire Line
+	3700 4100 3700 4200
+Wire Wire Line
+	3700 4200 3650 4200
+Wire Wire Line
+	1800 2000 1800 1900
+Wire Wire Line
+	1200 1650 1200 1900
+Wire Wire Line
+	4300 4150 3700 4150
+Connection ~ 3700 4150
+Wire Wire Line
+	4200 3800 4300 3800
+Wire Wire Line
+	4200 1450 2850 1450
+Wire Wire Line
+	1000 1450 1000 2150
+Wire Wire Line
+	1000 4300 1000 5850
+Connection ~ 1300 5850
+Wire Wire Line
+	4200 4500 4200 5850
+Connection ~ 3150 5850
+Wire Wire Line
+	3350 1450 3350 1550
+Connection ~ 3350 1450
 Wire Wire Line
 	3350 3150 3350 3050
-Connection ~ 3350 1450
-Wire Wire Line
-	3350 1550 3350 1450
-Connection ~ 3150 5850
+Wire Wire Line
+	2300 5600 2300 5450
+Wire Wire Line
+	2550 2750 3350 2750
+Wire Wire Line
+	1100 4000 1100 4100
 Wire Wire Line
 	4200 5850 1000 5850
-Wire Wire Line
-	4200 5850 4200 4500
-Connection ~ 1300 5850
-Wire Wire Line
-	1000 5850 1000 4300
-Wire Wire Line
-	1000 2150 1000 1450
-Wire Wire Line
-	2850 1450 4200 1450
-Wire Wire Line
-	4300 3800 4200 3800
-Connection ~ 3700 4150
-Wire Wire Line
-	4300 4150 3700 4150
-Wire Wire Line
-	1200 1650 1200 1900
-Wire Wire Line
-	1800 1900 1800 2000
-Wire Wire Line
-	3650 4200 3700 4200
-Wire Wire Line
-	3700 4200 3700 4100
-Wire Wire Line
-	3700 4100 3650 4100
-Wire Wire Line
-	1000 2550 1000 4000
-Wire Wire Line
-	1200 1650 1300 1650
-Connection ~ 2550 4000
-Wire Wire Line
-	2550 4000 2550 3750
-Connection ~ 1700 3800
-Wire Wire Line
-	1700 3800 1200 3800
-Wire Wire Line
-	1200 3800 1200 3250
-Wire Wire Line
-	2300 5600 2100 5600
-Wire Wire Line
-	740  4200 1100 4200
-Wire Wire Line
-	1000 4300 740  4300
-Wire Wire Line
-	1100 4200 1100 4300
-Connection ~ 2100 4000
-Wire Wire Line
-	1100 4300 2650 4300
-Wire Wire Line
-	2650 4000 1100 4000
-Connection ~ 2300 4300
-Connection ~ 3150 1450
-Wire Wire Line
-	2100 5600 2100 4950
-Wire Wire Line
-	2550 4550 2550 4300
-Connection ~ 2550 4300
-Wire Wire Line
-	1000 4000 740  4000
-Wire Wire Line
-	2100 4000 2100 4550
-Wire Wire Line
-	740  4100 1100 4100
-Wire Wire Line
-	1350 3350 1100 3350
-Wire Wire Line
-	1100 3350 1100 4100
-Connection ~ 1100 4000
-Wire Wire Line
-	2300 3350 2050 3350
-Connection ~ 2300 4300
-Wire Wire Line
-	1700 3000 1700 2750
-Connection ~ 3150 2750
-Wire Wire Line
-	1200 2850 1200 2750
-Connection ~ 1700 2750
-Wire Wire Line
-	1000 3900 1300 3900
-Wire Wire Line
-	1300 3900 1300 4550
-Connection ~ 1000 3900
-Wire Wire Line
-	1000 1450 1300 1450
-Wire Wire Line
-	2300 1650 2400 1650
-Wire Wire Line
-	2450 1450 2300 1450
-Wire Wire Line
-	2400 1650 2400 1900
-Wire Wire Line
-	2400 1900 1200 1900
-Connection ~ 1800 1900
-Wire Wire Line
-	3650 4000 4300 4000
-Wire Wire Line
-	4300 4300 3650 4300
-Wire Wire Line
-	4200 4500 4300 4500
-Wire Wire Line
-	3150 1400 3150 3600
-Wire Wire Line
-	4200 3800 4200 1450
-Wire Wire Line
-	2550 4950 2550 5100
-Wire Wire Line
-	2550 5100 3150 5100
-Connection ~ 3150 5100
-Wire Wire Line
-	3150 5850 3150 4700
-Wire Wire Line
-	1300 5950 1300 5050
-Wire Wire Line
-	2550 3350 2550 2750
-Connection ~ 2550 2750
-Wire Wire Line
-	1700 5850 1700 3700
-Connection ~ 1700 5850
-Wire Wire Line
-	3350 2850 3350 2750
-Wire Wire Line
-	3350 2750 1200 2750
-Wire Wire Line
-	3350 1850 3350 1750
-$Comp
-L GND #PWR022
+$Comp
+L GND #PWR04
 U 1 1 517A5C83
 P 3350 3150
-F 0 "#PWR022" H 3350 3150 30  0001 C CNN
+F 0 "#PWR04" H 3350 3150 30  0001 C CNN
 F 1 "GND" H 3350 3080 30  0001 C CNN
 	1    3350 3150
@@
 $EndComp
 $Comp
-L GND #PWR023
+L GND #PWR05
 U 1 1 517A5C80
 P 3350 1850
-F 0 "#PWR023" H 3350 1850 30  0001 C CNN
+F 0 "#PWR05" H 3350 1850 30  0001 C CNN
 F 1 "GND" H 3350 1780 30  0001 C CNN
 	1    3350 1850
@@
 $EndComp
 $Comp
-L VCC #PWR024
+L VCC #PWR06
 U 1 1 517A5B06
-P 3150 1400
-F 0 "#PWR024" H 3150 1500 30  0001 C CNN
-F 1 "VCC" H 3150 1500 30  0000 C CNN
-	1    3150 1400
+P 3150 1350
+F 0 "#PWR06" H 3150 1525 50  0001 C CNN
+F 1 "VCC" H 3150 1450 50  0000 C CNN
+	1    3150 1350
 	1    0    0    -1
 $EndComp
@@
 TXD
 $Comp
-L GND #PWR025
+L GND #PWR07
 U 1 1 517A5A68
 P 1300 5950
-F 0 "#PWR025" H 1300 5950 30  0001 C CNN
+F 0 "#PWR07" H 1300 5950 30  0001 C CNN
 F 1 "GND" H 1300 5880 30  0001 C CNN
 	1    1300 5950
@@
 $EndComp
 $Comp
-L GND #PWR026
+L GND #PWR08
 U 1 1 517A5A11
 P 1800 2000
-F 0 "#PWR026" H 1800 2000 30  0001 C CNN
+F 0 "#PWR08" H 1800 2000 30  0001 C CNN
 F 1 "GND" H 1800 1930 30  0001 C CNN
 	1    1800 2000
@@
 $EndComp
 $Comp
-L BRIDGE D301
-U 1 1 515DFB7E
-P 1350 3000
-F 0 "D301" H 1700 3500 50  0000 C CNN
-F 1 "BRIDGE" H 1700 3350 50  0000 C CNN
-	1    1350 3000
-	0    1    1    0
-$EndComp
-$Comp
-L ZD D302
-U 1 1 515DFFBA
-P 1200 3050
-F 0 "D302" H 1200 3150 50  0000 C CNN
-F 1 "P6SMB" H 1200 2950 50  0000 C CNN
-	1    1200 3050
-	0    -1   -1   0
-$EndComp
-$Comp
-L R R302
+L R R301
 U 1 1 5155E63E
 P 2100 4750
-F 0 "R302" H 2150 4850 50  0000 L CNN
+F 0 "R301" H 2150 4850 50  0000 L CNN
 F 1 "120R" H 2000 4750 50  0000 L CNN
 F 2 "~" H 2200 4740 50  0001 L CNN
@@
 $EndComp
 $Comp
-L R R301
+L R R302
 U 1 1 5155A27F
 P 2550 3550
-F 0 "R301" H 2600 3650 50  0000 L CNN
+F 0 "R302" H 2600 3650 50  0000 L CNN
 F 1 "390R" H 2450 3550 50  0000 L CNN
 F 2 "~" H 2650 3540 50  0001 L CNN

Commit message: - updated roomthermostate schematics - added hardware README
Parts:
- renumbered C301 to C23, C302 to C24, F302 to F1, F301 to F2, J301 to J1, J302 to J2, J303 to J3, J304 to J4, J305 to JP2, R304 to R14, R301 to R15, R302 to R16, R303 to R17, U301 to U6, U302 to U7
Changed lines of the file:
@@
-EESchema Schematic File Version 2  date So 05 Mai 2013 15:34:25 CEST
+EESchema Schematic File Version 2  date Sa 11 Mai 2013 12:24:20 CEST
+LIBS:connectors
+LIBS:display
+LIBS:encoder
+LIBS:ics_40xx
 LIBS:ics_controller_atmel
 LIBS:ics_misc
+LIBS:ics_opamp
+LIBS:ics_opto
+LIBS:ics_peripheral
 LIBS:ics_regulator
 LIBS:power
+LIBS:relays
+LIBS:sensors
 LIBS:standard
-LIBS:connectors
-LIBS:ics_peripheral
-LIBS:display
-LIBS:buscom-cache
-EELAYER 24  0
+LIBS:transformer
+LIBS:transistors
+LIBS:roomthermostate-cache
+EELAYER 25  0
 EELAYER END
 $Descr A4 11700 8267
-Sheet 3 3
+encoding utf-8
+Sheet 2 2
 Title ""
-Date "5 may 2013"
+Date "11 may 2013"
 Rev ""
 Comp ""
@@
 	4200 5850 1000 5850
 $Comp
-L GND #PWR04
+L GND #PWR28
 U 1 1 517A5C83
 P 3350 3150
-F 0 "#PWR04" H 3350 3150 30  0001 C CNN
+F 0 "#PWR28" H 3350 3150 30  0001 C CNN
 F 1 "GND" H 3350 3080 30  0001 C CNN
 	1    3350 3150
@@
 $EndComp
 $Comp
-L GND #PWR05
+L GND #PWR27
 U 1 1 517A5C80
 P 3350 1850
-F 0 "#PWR05" H 3350 1850 30  0001 C CNN
+F 0 "#PWR27" H 3350 1850 30  0001 C CNN
 F 1 "GND" H 3350 1780 30  0001 C CNN
 	1    3350 1850
@@
 $EndComp
 $Comp
-L C C301
+L C C23
 U 1 1 517A5C6F
 P 3350 1650
-F 0 "C301" H 3400 1700 50  0000 L CNN
+F 0 "C23" H 3400 1700 50  0000 L CNN
 F 1 "2,2uF" H 3350 1550 40  0000 C CNN
 F 4 "~" H 3150 1490 50  0001 L CNN "Voltage"
@@
 $EndComp
 $Comp
-L C C302
+L C C24
 U 1 1 517A5C42
 P 3350 2950
-F 0 "C302" H 3400 3000 50  0000 L CNN
+F 0 "C24" H 3400 3000 50  0000 L CNN
 F 1 "100nF" H 3350 2850 40  0000 C CNN
 F 4 "~" H 3150 2790 50  0001 L CNN "Voltage"
@@
 $EndComp
 $Comp
-L VCC #PWR06
+L VCC #PWR26
 U 1 1 517A5B06
 P 3150 1350
-F 0 "#PWR06" H 3150 1525 50  0001 C CNN
+F 0 "#PWR26" H 3150 1525 50  0001 C CNN
 F 1 "VCC" H 3150 1450 50  0000 C CNN
 	1    3150 1350
@@
 TXD
 $Comp
-L GND #PWR07
+L GND #PWR24
 U 1 1 517A5A68
 P 1300 5950
-F 0 "#PWR07" H 1300 5950 30  0001 C CNN
+F 0 "#PWR24" H 1300 5950 30  0001 C CNN
 F 1 "GND" H 1300 5880 30  0001 C CNN
 	1    1300 5950
@@
 $EndComp
 $Comp
-L GND #PWR08
+L GND #PWR25
 U 1 1 517A5A11
 P 1800 2000
-F 0 "#PWR08" H 1800 2000 30  0001 C CNN
+F 0 "#PWR25" H 1800 2000 30  0001 C CNN
 F 1 "GND" H 1800 1930 30  0001 C CNN
 	1    1800 2000
@@
 $EndComp
 $Comp
-L FUSE F302
+L FUSE F1
 U 1 1 517A45B7
 P 1000 2350
-F 0 "F302" H 1000 2450 50  0000 C CNN
+F 0 "F1" H 1000 2450 50  0000 C CNN
 F 1 "FUSE" H 1000 2250 50  0000 C CNN
 	1    1000 2350
@@
 $EndComp
 $Comp
-L FUSE F301
+L FUSE F2
 U 1 1 517A4454
 P 2650 1450
-F 0 "F301" H 2650 1550 50  0000 C CNN
+F 0 "F2" H 2650 1550 50  0000 C CNN
 F 1 "FUSE" H 2650 1350 50  0000 C CNN
 	1    2650 1450
@@
 +24
 $Comp
-L CONN_1 J301
+L CONN_1 J1
 U 1 1 51673922
 P 640 4000
-F 0 "J301" H 640 4040 40  0000 C CNN
-F 1 "CONN_1" H 550 3970 25  0000 C CNN
+F 0 "J1" H 640 4040 40  0000 C CNN
+F 1 "CONN_1" H 550 3970 25  0001 C CNN
 	1    640  4000
 	-1   0    0    -1
 $EndComp
 $Comp
-L CONN_1 J302
+L CONN_1 J2
 U 1 1 5167391D
 P 640 4100
-F 0 "J302" H 640 4140 40  0000 C CNN
-F 1 "CONN_1" H 550 4070 25  0000 C CNN
+F 0 "J2" H 640 4140 40  0000 C CNN
+F 1 "CONN_1" H 550 4070 25  0001 C CNN
 	1    640  4100
 	-1   0    0    -1
 $EndComp
 $Comp
-L CONN_1 J303
+L CONN_1 J3
 U 1 1 5167391A
 P 640 4200
-F 0 "J303" H 640 4240 40  0000 C CNN
-F 1 "CONN_1" H 550 4170 25  0000 C CNN
+F 0 "J3" H 640 4240 40  0000 C CNN
+F 1 "CONN_1" H 550 4170 25  0001 C CNN
 	1    640  4200
 	-1   0    0    -1
 $EndComp
 $Comp
-L CONN_1 J304
+L CONN_1 J4
 U 1 1 51673909
 P 640 4300
-F 0 "J304" H 640 4340 40  0000 C CNN
-F 1 "CONN_1" H 550 4270 25  0000 C CNN
+F 0 "J4" H 640 4340 40  0000 C CNN
+F 1 "CONN_1" H 550 4270 25  0001 C CNN
 	1    640  4300
 	-1   0    0    -1
 $EndComp
 $Comp
-L VARISTOR R304
+L VARISTOR R14
 U 1 1 515FF5C8
 P 1300 4800
-F 0 "R304" H 1170 4710 50  0000 C CNN
+F 0 "R14" H 1170 4710 50  0000 C CNN
 F 1 "VARISTOR" H 1300 4800 40  0000 C CNN
 F 2 "~" H 1400 4790 50  0001 L CNN
@@
 $EndComp
 $Comp
-L R R301
+L R R15
 U 1 1 5155E63E
 P 2100 4750
-F 0 "R301" H 2150 4850 50  0000 L CNN
+F 0 "R15" H 2150 4850 50  0000 L CNN
 F 1 "120R" H 2000 4750 50  0000 L CNN
 F 2 "~" H 2200 4740 50  0001 L CNN
@@
 $EndComp
 $Comp
-L JUMPER J305
+L JUMPER JP2
 U 1 1 5155E40C
 P 2300 5300
-F 0 "J305" H 2250 5450 60  0000 C CNN
-F 1 "JUMPER" H 2300 5150 60  0000 C CNN
+F 0 "JP2" H 2250 5450 60  0000 C CNN
+F 1 "JUMPER" H 2300 5150 60  0001 C CNN
 	1    2300 5300
 	0    1    1    0
 $EndComp
 $Comp
-L AM1S-2405 U301
+L AM1S-2405 U6
 U 1 1 5155B854
 P 1800 1550
-F 0 "U301" H 1800 1550 40  0000 C CNN
+F 0 "U6" H 1800 1550 40  0000 C CNN
 F 1 "AM1S-2405" H 1800 1350 40  0000 C CNN
 F 2 "MODULE" H 1800 1550 40  0001 C CNN
@@
 $EndComp
 $Comp
-L MAX487 U302
+L MAX487 U7
 U 1 1 5155AE3E
 P 3150 4150
-F 0 "U302" H 3400 4550 60  0000 C CNN
+F 0 "U7" H 3400 4550 60  0000 C CNN
 F 1 "MAX487" H 2950 3750 60  0000 C CNN
 F 2 "SSOP28" H 3000 4700 40  0001 C CNN
@@
 $EndComp
 $Comp
-L R R303
+L R R17
 U 1 1 5155A28E
 P 2550 4750
-F 0 "R303" H 2600 4850 50  0000 L CNN
+F 0 "R17" H 2600 4850 50  0000 L CNN
 F 1 "390R" H 2450 4750 50  0000 L CNN
 F 2 "~" H 2650 4740 50  0001 L CNN
@@
 $EndComp
 $Comp
-L R R302
+L R R16
 U 1 1 5155A27F
 P 2550 3550
-F 0 "R302" H 2600 3650 50  0000 L CNN
+F 0 "R16" H 2600 3650 50  0000 L CNN
 F 1 "390R" H 2450 3550 50  0000 L CNN
 F 2 "~" H 2650 3540 50  0001 L CNN

Commit message: new schematic symbols used
Parts:
- removed U7: MAX487, SSOP28, symbol MAX487
- added U?: MAX487, SSOP28, symbol MAX487
Changed lines of the file:
@@
-EESchema Schematic File Version 2  date Di 02 Jul 2013 07:38:50 CEST
+EESchema Schematic File Version 2  date Fr 01 Nov 2013 16:45:02 CET
 LIBS:connectors
 LIBS:display
@@
 Sheet 2 2
 Title ""
-Date "2 jul 2013"
+Date "1 nov 2013"
 Rev ""
 Comp ""
@@
 Comment4 ""
 $EndDescr
+$Comp
+L MAX487 U?
+U 1 1 5273CC68
+P 3150 4150
+F 0 "U?" H 2900 4550 50  0000 C CNN
+F 1 "MAX487" H 3350 3750 50  0000 C CNN
+F 2 "SSOP28" H 3000 3750 25  0001 C CNN
+	1    3150 4150
+	-1   0    0    -1
+$EndComp
 Wire Wire Line
 	3150 1350 3150 3600
@@
 $EndComp
 $Comp
-L MAX487 U7
-U 1 1 5155AE3E
-P 3150 4150
-F 0 "U7" H 3400 4550 60  0000 C CNN
-F 1 "MAX487" H 2950 3750 60  0000 C CNN
-F 2 "SSOP28" H 3000 4700 40  0001 C CNN
-	1    3150 4150
-	-1   0    0    -1
-$EndComp
-$Comp

Commit message: Schematic changes: - TXEN now on PD4 - Temperature sensor power is switchable - LCD Reset added - CS of EEP and LCD switched
Parts:
- removed R16, R17: 390R, ~, symbol R
- J10: renamed from J1; value CONN_1 -> +24V
- J11: renamed from J2; value CONN_1 -> BUS_A
- J12: renamed from J3; value CONN_1 -> BUS_B
- J13: renamed from J4; value CONN_1 -> GND
- gave numbers to parts that had none: 1
- renumbered C23 to C24, C24 to C25, R14 to R18, R15 to R19
Connections:
- wire segments 51 -> 46
Changed lines of the file:
@@
-EESchema Schematic File Version 2  date Fr 01 Nov 2013 16:45:02 CET
+EESchema Schematic File Version 2  date Mo 30 Dez 2013 09:55:07 CET
 LIBS:connectors
 LIBS:display
@@
 Sheet 2 2
 Title ""
-Date "1 nov 2013"
+Date "30 dec 2013"
 Rev ""
 Comp ""
@@
 Comment4 ""
 $EndDescr
-$Comp
-L MAX487 U?
+Wire Wire Line
+	3150 2750 3350 2750
+Wire Wire Line
+	4200 5850 1000 5850
+Wire Wire Line
+	1100 4000 1100 4100
+Wire Wire Line
+	2300 5450 2300 5600
+Wire Wire Line
+	3350 3150 3350 3050
+Connection ~ 3350 1450
+Wire Wire Line
+	3350 1450 3350 1550
+Connection ~ 3150 5850
+Wire Wire Line
+	4200 5850 4200 4500
+Connection ~ 1300 5850
+Wire Wire Line
+	1000 5850 1000 4300
+Wire Wire Line
+	1000 2150 1000 1450
+Wire Wire Line
+	2850 1450 4200 1450
+Wire Wire Line
+	4300 3800 4200 3800
+Connection ~ 3700 4150
+Wire Wire Line
+	4300 4150 3700 4150
+Wire Wire Line
+	1200 1650 1200 1900
+Wire Wire Line
+	1800 2000 1800 1900
+Wire Wire Line
+	3650 4200 3700 4200
+Wire Wire Line
+	3700 4200 3700 4100
+Wire Wire Line
+	3700 4100 3650 4100
+Wire Wire Line
+	1000 2550 1000 4000
+Wire Wire Line
+	1200 1650 1300 1650
+Wire Wire Line
+	2300 5600 2100 5600
+Wire Wire Line
+	740  4200 1100 4200
+Wire Wire Line
+	1000 4300 740  4300
+Wire Wire Line
+	1100 4200 1100 4300
+Connection ~ 2100 4000
+Wire Wire Line
+	1100 4300 2650 4300
+Wire Wire Line
+	1100 4000 2650 4000
+Connection ~ 2300 4300
+Wire Wire Line
+	2100 5600 2100 4950
+Wire Wire Line
+	1000 4000 740  4000
+Wire Wire Line
+	2100 4000 2100 4550
+Wire Wire Line
+	1100 4100 740  4100
+Connection ~ 2300 4300
+Connection ~ 3150 2750
+Wire Wire Line
+	1000 3900 1300 3900
+Wire Wire Line
+	1300 3900 1300 4550
+Connection ~ 1000 3900
+Wire Wire Line
+	1000 1450 1300 1450
+Wire Wire Line
+	2300 1650 2400 1650
+Wire Wire Line
+	2450 1450 2300 1450
+Wire Wire Line
+	2400 1650 2400 1900
+Wire Wire Line
+	2400 1900 1200 1900
+Connection ~ 1800 1900
+Wire Wire Line
+	3650 4000 4300 4000
+Wire Wire Line
+	4300 4300 3650 4300
+Wire Wire Line
+	4200 4500 4300 4500
+Wire Wire Line
+	4200 3800 4200 1450
+Wire Wire Line
+	3150 5850 3150 4700
+Wire Wire Line
+	1300 5950 1300 5050
+Wire Wire Line
+	3350 2750 3350 2850
+Wire Wire Line
+	3350 1850 3350 1750
+Wire Wire Line
+	2300 5150 2300 4300
+Connection ~ 3150 1450
+Wire Wire Line
+	3150 1350 3150 3600
+$Comp
+L MAX487 U7
 U 1 1 5273CC68
 P 3150 4150
-F 0 "U?" H 2900 4550 50  0000 C CNN
+F 0 "U7" H 2900 4550 50  0000 C CNN
 F 1 "MAX487" H 3350 3750 50  0000 C CNN
 F 2 "SSOP28" H 3000 3750 25  0001 C CNN
@@
 	-1   0    0    -1
 $EndComp
-Wire Wire Line
-	3150 1350 3150 3600
-Connection ~ 3150 1450
-Wire Wire Line
-	2300 5150 2300 4300
-Wire Wire Line
-	3350 1850 3350 1750
-Wire Wire Line
-	3350 2850 3350 2750
-Wire Wire Line
-	2550 3350 2550 2750
-Wire Wire Line
-	1300 5950 1300 5050
-Wire Wire Line
-	3150 5850 3150 4700
-Connection ~ 3150 5100
-Wire Wire Line
-	3150 5100 2550 5100
-Wire Wire Line
-	2550 5100 2550 4950
-Wire Wire Line
-	4200 3800 4200 1450
-Wire Wire Line
-	4300 4500 4200 4500
-Wire Wire Line
-	4300 4300 3650 4300
-Wire Wire Line
-	3650 4000 4300 4000
-Connection ~ 1800 1900
-Wire Wire Line
-	2400 1900 1200 1900
-Wire Wire Line
-	2400 1900 2400 1650
-Wire Wire Line
-	2450 1450 2300 1450
-Wire Wire Line
-	2400 1650 2300 1650
-Wire Wire Line
-	1300 1450 1000 1450
-Connection ~ 1000 3900
-Wire Wire Line
-	1300 4550 1300 3900
-Wire Wire Line
-	1300 3900 1000 3900
-Connection ~ 3150 2750
-Connection ~ 2300 4300
-Wire Wire Line
-	740  4100 1100 4100
-Wire Wire Line
-	2100 4000 2100 4550
-Wire Wire Line
-	740  4000 1000 4000
-Connection ~ 2550 4300
-Wire Wire Line
-	2550 4550 2550 4300
-Wire Wire Line
-	2100 4950 2100 5600
-Connection ~ 2300 4300
-Wire Wire Line
-	2650 4000 1100 4000
-Wire Wire Line
-	2650 4300 1100 4300
-Connection ~ 2100 4000
-Wire Wire Line
-	1100 4300 1100 4200
-Wire Wire Line
-	740  4300 1000 4300
-Wire Wire Line
-	1100 4200 740  4200
-Wire Wire Line
-	2100 5600 2300 5600
-Wire Wire Line
-	2550 4000 2550 3750
-Connection ~ 2550 4000
-Wire Wire Line
-	1300 1650 1200 1650
-Wire Wire Line
-	1000 4000 1000 2550
-Wire Wire Line
-	3650 4100 3700 4100
-Wire Wire Line
-	3700 4100 3700 4200
-Wire Wire Line
-	3700 4200 3650 4200
-Wire Wire Line
-	1800 2000 1800 1900
-Wire Wire Line
-	1200 1650 1200 1900
-Wire Wire Line
-	4300 4150 3700 4150
-Connection ~ 3700 4150
-Wire Wire Line
-	4200 3800 4300 3800
-Wire Wire Line
-	4200 1450 2850 1450
-Wire Wire Line
-	1000 1450 1000 2150
-Wire Wire Line
-	1000 4300 1000 5850
-Connection ~ 1300 5850
-Wire Wire Line
-	4200 4500 4200 5850
-Connection ~ 3150 5850
-Wire Wire Line
-	3350 1450 3350 1550
-Connection ~ 3350 1450
-Wire Wire Line
-	3350 3150 3350 3050
-Wire Wire Line
-	2300 5600 2300 5450
-Wire Wire Line
-	2550 2750 3350 2750
-Wire Wire Line
-	1100 4000 1100 4100
-Wire Wire Line
-	4200 5850 1000 5850
-$Comp
-L GND #PWR024
+$Comp
+L GND #PWR027
 U 1 1 517A5C83
 P 3350 3150
-F 0 "#PWR024" H 3350 3150 30  0001 C CNN
+F 0 "#PWR027" H 3350 3150 30  0001 C CNN
 F 1 "GND" H 3350 3080 30  0001 C CNN
 	1    3350 3150
@@
 $EndComp
 $Comp
-L GND #PWR025
+L GND #PWR028
 U 1 1 517A5C80
 P 3350 1850
-F 0 "#PWR025" H 3350 1850 30  0001 C CNN
+F 0 "#PWR028" H 3350 1850 30  0001 C CNN
 F 1 "GND" H 3350 1780 30  0001 C CNN
 	1    3350 1850
@@
 $EndComp
 $Comp
-L C C23
+L C C24
 U 1 1 517A5C6F
 P 3350 1650
-F 0 "C23" H 3400 1700 50  0000 L CNN
+F 0 "C24" H 3400 1700 50  0000 L CNN
 F 1 "2,2uF" H 3350 1550 40  0000 C CNN
 F 4 "~" H 3150 1490 50  0001 L CNN "Voltage"
@@
 $EndComp
 $Comp
-L C C24
+L C C25
 U 1 1 517A5C42
 P 3350 2950
-F 0 "C24" H 3400 3000 50  0000 L CNN
+F 0 "C25" H 3400 3000 50  0000 L CNN
 F 1 "100nF" H 3350 2850 40  0000 C CNN
 F 4 "~" H 3150 2790 50  0001 L CNN "Voltage"
@@
 $EndComp
 $Comp
-L VCC #PWR026
+L VCC #PWR029
 U 1 1 517A5B06
 P 3150 1350
-F 0 "#PWR026" H 3150 1525 50  0001 C CNN
+F 0 "#PWR029" H 3150 1525 50  0001 C CNN
 F 1 "VCC" H 3150 1450 50  0000 C CNN
 	1    3150 1350
@@
 TXD
 $Comp
-L GND #PWR027
+L GND #PWR030
 U 1 1 517A5A68
 P 1300 5950
-F 0 "#PWR027" H 1300 5950 30  0001 C CNN
+F 0 "#PWR030" H 1300 5950 30  0001 C CNN
 F 1 "GND" H 1300 5880 30  0001 C CNN
 	1    1300 5950
@@
 $EndComp
 $Comp
-L GND #PWR028
+L GND #PWR031
 U 1 1 517A5A11
 P 1800 2000
-F 0 "#PWR028" H 1800 2000 30  0001 C CNN
+F 0 "#PWR031" H 1800 2000 30  0001 C CNN
 F 1 "GND" H 1800 1930 30  0001 C CNN
 	1    1800 2000
@@
 +24
 $Comp
-L CONN_1 J1
+L CONN_1 J10
 U 1 1 51673922
 P 640 4000
-F 0 "J1" H 640 4040 40  0000 C CNN
-F 1 "CONN_1" H 550 3970 25  0001 C CNN
+F 0 "J10" H 640 4040 40  0000 C CNN
+F 1 "+24V" H 550 3970 25  0001 C CNN
 	1    640  4000
 	-1   0    0    -1
 $EndComp
 $Comp
-L CONN_1 J2
+L CONN_1 J11
 U 1 1 5167391D
 P 640 4100
-F 0 "J2" H 640 4140 40  0000 C CNN
-F 1 "CONN_1" H 550 4070 25  0001 C CNN
+F 0 "J11" H 640 4140 40  0000 C CNN
+F 1 "BUS_A" H 550 4070 25  0001 C CNN
 	1    640  4100
 	-1   0    0    -1
 $EndComp
 $Comp
-L CONN_1 J3
+L CONN_1 J12
 U 1 1 5167391A
 P 640 4200
-F 0 "J3" H 640 4240 40  0000 C CNN
-F 1 "CONN_1" H 550 4170 25  0001 C CNN
+F 0 "J12" H 640 4240 40  0000 C CNN
+F 1 "BUS_B" H 550 4170 25  0001 C CNN
 	1    640  4200
 	-1   0    0    -1
 $EndComp
 $Comp
-L CONN_1 J4
+L CONN_1 J13
 U 1 1 51673909
 P 640 4300
-F 0 "J4" H 640 4340 40  0000 C CNN
-F 1 "CONN_1" H 550 4270 25  0001 C CNN
+F 0 "J13" H 640 4340 40  0000 C CNN
+F 1 "GND" H 550 4270 25  0001 C CNN
 	1    640  4300
 	-1   0    0    -1
 $EndComp
 $Comp
-L VARISTOR R14
+L VARISTOR R18
 U 1 1 515FF5C8
 P 1300 4800
-F 0 "R14" H 1170 4710 50  0000 C CNN
+F 0 "R18" H 1170 4710 50  0000 C CNN
 F 1 "VARISTOR" H 1300 4800 40  0000 C CNN
 F 2 "~" H 1400 4790 50  0001 L CNN
@@
 $EndComp
 $Comp
-L R R15
+L R R19
 U 1 1 5155E63E
 P 2100 4750
-F 0 "R15" H 2150 4850 50  0000 L CNN
+F 0 "R19" H 2150 4850 50  0000 L CNN
 F 1 "120R" H 2000 4750 50  0000 L CNN
 F 2 "~" H 2200 4740 50  0001 L CNN
@@
 	1    0    0    -1
 $EndComp
-$Comp
-L R R17
-U 1 1 5155A28E
-P 2550 4750
-F 0 "R17" H 2600 4850 50  0000 L CNN
-F 1 "390R" H 2450 4750 50  0000 L CNN
-F 2 "~" H 2650 4740 50  0001 L CNN
-F 3 "~" H 2650 4680 50  0001 L CNN
-	1    2550 4750
-	0    1    1    0
-$EndComp
-$Comp
-L R R16
-U 1 1 5155A27F
-P 2550 3550
-F 0 "R16" H 2600 3650 50  0000 L CNN
-F 1 "390R" H 2450 3550 50  0000 L CNN
-F 2 "~" H 2650 3540 50  0001 L CNN
-F 3 "~" H 2650 3480 50  0001 L CNN
-	1    2550 3550
-	0    1    1    0
-$EndComp
 $EndSCHEMATC
