File: hw/roomthermostat/businterface.sch (KiCad schematic (older format))
At the start: 13 parts, among them J10 +24V, J11 BUS_A, J12 BUS_B, J13 GND, U6 AM1S-2405, U7 MAX487

Commit message: Use bus-module_atmega328 instead of single atmega324 controller.
Parts:
- R18: symbol VARISTOR -> Varistor
Changed lines of the file:
@@
-EESchema Schematic File Version 2  date Mo 30 Dez 2013 09:55:07 CET
+EESchema Schematic File Version 2
+LIBS:roomthermostate-rescue
 LIBS:connectors
 LIBS:display
@@
 LIBS:transformer
 LIBS:transistors
+LIBS:modules
 LIBS:roomthermostate-cache
-EELAYER 25  0
+EELAYER 25 0
 EELAYER END
-$Descr A4 11700 8267
+$Descr A4 11693 8268
 encoding utf-8
 Sheet 2 2
@@
 F 1 "MAX487" H 3350 3750 50  0000 C CNN
 F 2 "SSOP28" H 3000 3750 25  0001 C CNN
+F 3 "" H 3150 4150 60  0001 C CNN
 	1    3150 4150
 	-1   0    0    -1
 $EndComp
 $Comp
-L GND #PWR027
+L GND-RESCUE-roomthermostate #PWR027
 U 1 1 517A5C83
 P 3350 3150
 F 0 "#PWR027" H 3350 3150 30  0001 C CNN
 F 1 "GND" H 3350 3080 30  0001 C CNN
+F 2 "" H 3350 3150 60  0001 C CNN
+F 3 "" H 3350 3150 60  0001 C CNN
 	1    3350 3150
 	1    0    0    -1
 $EndComp
 $Comp
-L GND #PWR028
+L GND-RESCUE-roomthermostate #PWR028
 U 1 1 517A5C80
 P 3350 1850
 F 0 "#PWR028" H 3350 1850 30  0001 C CNN
 F 1 "GND" H 3350 1780 30  0001 C CNN
+F 2 "" H 3350 1850 60  0001 C CNN
+F 3 "" H 3350 1850 60  0001 C CNN
 	1    3350 1850
 	1    0    0    -1
@@
 F 0 "C24" H 3400 1700 50  0000 L CNN
 F 1 "2,2uF" H 3350 1550 40  0000 C CNN
+F 2 "" H 3350 1650 60  0001 C CNN
+F 3 "" H 3350 1650 60  0001 C CNN
 F 4 "~" H 3150 1490 50  0001 L CNN "Voltage"
 F 5 "~" H 3150 1430 50  0001 L CNN "Tolerance"
@@
 F 0 "C25" H 3400 3000 50  0000 L CNN
 F 1 "100nF" H 3350 2850 40  0000 C CNN
+F 2 "" H 3350 2950 60  0001 C CNN
+F 3 "" H 3350 2950 60  0001 C CNN
 F 4 "~" H 3150 2790 50  0001 L CNN "Voltage"
 F 5 "~" H 3150 2730 50  0001 L CNN "Tolerance"
@@
 F 0 "#PWR029" H 3150 1525 50  0001 C CNN
 F 1 "VCC" H 3150 1450 50  0000 C CNN
+F 2 "" H 3150 1350 60  0001 C CNN
+F 3 "" H 3150 1350 60  0001 C CNN
 	1    3150 1350
 	1    0    0    -1
@@
 TXD
 $Comp
-L GND #PWR030
+L GND-RESCUE-roomthermostate #PWR030
 U 1 1 517A5A68
 P 1300 5950
 F 0 "#PWR030" H 1300 5950 30  0001 C CNN
 F 1 "GND" H 1300 5880 30  0001 C CNN
+F 2 "" H 1300 5950 60  0001 C CNN
+F 3 "" H 1300 5950 60  0001 C CNN
 	1    1300 5950
 	1    0    0    -1
 $EndComp
 $Comp
-L GND #PWR031
+L GND-RESCUE-roomthermostate #PWR031
 U 1 1 517A5A11
 P 1800 2000
 F 0 "#PWR031" H 1800 2000 30  0001 C CNN
 F 1 "GND" H 1800 1930 30  0001 C CNN
+F 2 "" H 1800 2000 60  0001 C CNN
+F 3 "" H 1800 2000 60  0001 C CNN
 	1    1800 2000
 	1    0    0    -1
@@
 F 0 "F1" H 1000 2450 50  0000 C CNN
 F 1 "FUSE" H 1000 2250 50  0000 C CNN
+F 2 "" H 1000 2350 60  0001 C CNN
+F 3 "" H 1000 2350 60  0001 C CNN
 	1    1000 2350
 	0    1    1    0
@@
 F 0 "F2" H 2650 1550 50  0000 C CNN
 F 1 "FUSE" H 2650 1350 50  0000 C CNN
+F 2 "" H 2650 1450 60  0001 C CNN
+F 3 "" H 2650 1450 60  0001 C CNN
 	1    2650 1450
 	1    0    0    -1
@@
 F 0 "J10" H 640 4040 40  0000 C CNN
 F 1 "+24V" H 550 3970 25  0001 C CNN
+F 2 "" H 640 4000 60  0001 C CNN
+F 3 "" H 640 4000 60  0001 C CNN
 	1    640  4000
 	-1   0    0    -1
@@
 F 0 "J11" H 640 4140 40  0000 C CNN
 F 1 "BUS_A" H 550 4070 25  0001 C CNN
+F 2 "" H 640 4100 60  0001 C CNN
+F 3 "" H 640 4100 60  0001 C CNN
 	1    640  4100
 	-1   0    0    -1
@@
 F 0 "J12" H 640 4240 40  0000 C CNN
 F 1 "BUS_B" H 550 4170 25  0001 C CNN
+F 2 "" H 640 4200 60  0001 C CNN
+F 3 "" H 640 4200 60  0001 C CNN
 	1    640  4200
 	-1   0    0    -1
@@
 F 0 "J13" H 640 4340 40  0000 C CNN
 F 1 "GND" H 550 4270 25  0001 C CNN
+F 2 "" H 640 4300 60  0001 C CNN
+F 3 "" H 640 4300 60  0001 C CNN
 	1    640  4300
 	-1   0    0    -1
 $EndComp
 $Comp
-L VARISTOR R18
+L Varistor R18
 U 1 1 515FF5C8
 P 1300 4800
@@
 F 0 "JP2" H 2250 5450 60  0000 C CNN
 F 1 "JUMPER" H 2300 5150 60  0001 C CNN
+F 2 "" H 2300 5300 60  0001 C CNN
+F 3 "" H 2300 5300 60  0001 C CNN
 	1    2300 5300
 	0    1    1    0
