File: hw/motor_switch_3pole/bus_atmega328_basic.sch (KiCad schematic (older format))
At the start: 26 parts, among them J3 CONN-ISP-6, J4 CONN_1, J5 CONN_1, J6 CONN_1, J7 CONN_1, U1 25LC256, U2 ATMEGA328-TQFP32, U3 7,3728MHz, U4 MAX487ECSA, U5 AM1S-2403

Commit message: Final revision 1 files of motor_switch_3pole added. Prototype PCBs of this revision have been ordered
Parts:
- C7: value 47µF / 4V -> 100µF / 6V; footprint Capacitors_SMD:C_0805 -> Capacitors_SMD:C_1206
- J4: value CONN_1 -> WAGO 243-723
- J5: value CONN_1 -> WAGO 243-724
- J6: value CONN_1 -> WAGO 243-721
- J7: value CONN_1 -> WAGO 243-722
- U5: value AM1S-2403 -> AM1S-2405
Changed lines of the file:
@@
 encoding utf-8
 Sheet 2 2
-Title "bus_atmega328_basic"
-Date "2016-07-16"
+Title "motor switch 3pole (bus_atmega328_basic)"
+Date "2016-09-06"
 Rev "1"
 Comp "KoeWiBa"
@@
 P 10150 2500
 F 0 "J4" H 10150 2575 50  0000 C CNN
-F 1 "CONN_1" H 10150 2425 25  0000 C CNN
+F 1 "WAGO 243-723" H 10150 2450 25  0000 C CNN
 F 2 "Connector_WAGO:WAGO_243" H 10150 2500 60  0001 C CNN
 F 3 "" H 10150 2500 60  0000 C CNN
@@
 P 10150 2700
 F 0 "J5" H 10150 2775 50  0000 C CNN
-F 1 "CONN_1" H 10150 2625 25  0000 C CNN
+F 1 "WAGO 243-724" H 10150 2650 25  0000 C CNN
 F 2 "Connector_WAGO:WAGO_243" H 10150 2700 60  0001 C CNN
 F 3 "" H 10150 2700 60  0000 C CNN
@@
 P 10150 2900
 F 0 "J6" H 10150 2975 50  0000 C CNN
-F 1 "CONN_1" H 10150 2825 25  0000 C CNN
+F 1 "WAGO 243-721" H 10150 2850 25  0000 C CNN
 F 2 "Connector_WAGO:WAGO_243" H 10150 2900 60  0001 C CNN
 F 3 "" H 10150 2900 60  0000 C CNN
@@
 P 10150 3100
 F 0 "J7" H 10150 3175 50  0000 C CNN
-F 1 "CONN_1" H 10150 3025 25  0000 C CNN
+F 1 "WAGO 243-722" H 10150 3050 25  0000 C CNN
 F 2 "Connector_WAGO:WAGO_243" H 10150 3100 60  0001 C CNN
 F 3 "" H 10150 3100 60  0000 C CNN
@@
 P 8050 1300
 F 0 "U5" H 8050 1300 50  0000 C CNN
-F 1 "AM1S-2403" H 8050 1100 50  0000 C CNN
+F 1 "AM1S-2405" H 8050 1100 50  0000 C CNN
 F 2 "DCDC_Converter:AM1S-XXXX_SIL4" H 8050 1500 25  0001 C CNN
 F 3 "" H 7300 1300 25  0001 C CNN
@@
 P 7200 1300
 F 0 "C7" H 7250 1350 50  0000 L CNN
-F 1 "47µF / 4V" H 7200 1175 50  0000 C CNN
-F 2 "Capacitors_SMD:C_0805" H 7200 1300 60  0001 C CNN
+F 1 "100µF / 6V" H 7200 1175 50  0000 C CNN
+F 2 "Capacitors_SMD:C_1206" H 7200 1300 60  0001 C CNN
 F 3 "" H 7200 1300 60  0000 C CNN
 	1    7200 1300
