File: hw/pi2-base/pi2-base.sch (KiCad schematic (older format))
At the start: 36 parts, among them J1 WAGO 2081-1122, J10 BUS Pull-down, J11 JUMPER3, J12 JUMPER3, J13 Power LEDs, J14 JUMPER3, J15 JUMPER3, J16 JUMPER3, J17 JUMPER3, J2 WAGO 243 orange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

Commit message: Changed resistor values from 56k/100k to 10k/18k of voltage divider of TXD and CTS
Parts:
- R10, R9: value 100k -> 18k
- R6, R7: value 56k -> 10k
Changed lines of the file:
@@
 EESchema Schematic File Version 2
+LIBS:pi2-base-rescue
 LIBS:connectors
 LIBS:diodes
@@
 Sheet 1 5
 Title "pi2-base"
-Date "2016-12-11"
+Date "2017-02-10"
 Rev "1"
 Comp "KoeWiBa"
@@
 P 5800 3100
 F 0 "R6" H 6050 3150 50  0000 C CNN
-F 1 "56k" H 5800 3100 50  0000 C CNN
+F 1 "10k" H 5800 3100 50  0000 C CNN
 F 2 "Resistor:R_0805" H 5800 3100 60  0001 C CNN
 F 3 "" H 5800 3100 60  0000 C CNN
@@
 P 5800 3250
 F 0 "R7" H 6050 3300 50  0000 C CNN
-F 1 "56k" H 5800 3250 50  0000 C CNN
+F 1 "10k" H 5800 3250 50  0000 C CNN
 F 2 "Resistor:R_0805" H 5800 3250 60  0001 C CNN
 F 3 "" H 5800 3250 60  0000 C CNN
@@
 P 6100 3550
 F 0 "R9" H 6100 3450 50  0000 L CNN
-F 1 "100k" H 6100 3550 50  0000 C CNN
+F 1 "18k" H 6100 3550 50  0000 C CNN
 F 2 "Resistor:R_0805" H 6100 3550 60  0001 C CNN
 F 3 "" H 6100 3550 60  0000 C CNN
@@
 P 6300 3550
 F 0 "R10" H 6300 3650 50  0000 L CNN
-F 1 "100k" H 6300 3550 50  0000 C CNN
+F 1 "18k" H 6300 3550 50  0000 C CNN
 F 2 "Resistor:R_0805" H 6300 3550 60  0001 C CNN
 F 3 "" H 6300 3550 60  0000 C CNN
