File: hw/pi2-base/pi2-base.sch (KiCad schematic (older format))
At the start: 36 parts, among them J1 WAGO 2081-1122, J10 BUS Pull-down, J11 JUMPER3, J12 JUMPER3, J13 Power LEDs, J14 JUMPER3, J15 JUMPER3, J16 JUMPER3, J17 JUMPER3, J2 WAGO 243 orange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

Commit message: Fix: Silkscreen jumper description Fix: Relay pinout
Other:
- note added: "Do NOT use relays for 230V!\nIsolation for 230V not sufficient!"
Changed lines of the file:
@@
 EESchema Schematic File Version 2
+LIBS:pi2-base-rescue
 LIBS:connectors
 LIBS:diodes
@@
 LIBS:ics_peripheral
 LIBS:pi2-base-cache
-EELAYER 26 0
+EELAYER 25 0
 EELAYER END
 $Descr A4 11693 8268
@@
 Sheet 1 5
 Title "pi2-base"
-Date "2017-02-10"
-Rev "1"
+Date "2018-06-12"
+Rev "2"
 Comp "KoeWiBa"
 Comment1 "Base board for Raspberry Pi B2"
@@
 	1    0    0    -1
 $EndComp
+Text Notes 600  3100 0    50   ~ 0
+Do NOT use relays for 230V!\nIsolation for 230V not sufficient!
 $EndSCHEMATC

Commit message: Renamed Rev2 -> RevB Updated 3d footprints Replaced busmodule RevA with RevB symbol
Parts:
- removed MOD1: bus-module_atmega324, Modules:bus-module_atmega324, symbol bus-module_atmega324
- added MOD1: bus-module_atmega324_revB, symbol modules:bus-module_atmega324_revB
- F1: symbol FUSE -> standard:FUSE
- H1, H2, H3, H4: symbol HOLE -> standard:HOLE
- J1: symbol CONN_2X1 -> connectors:CONN_2X1
- J10, J13, J9: symbol JUMPER -> connectors:JUMPER
- J11, J12, J14, J15, J16, J17: symbol JUMPER3 -> connectors:JUMPER3
- J2, J3, J4, J5: symbol CONN_1X1 -> connectors:CONN_1X1
- J6, J7: symbol CONN_3X1 -> connectors:CONN_3X1
- J8: symbol CONN_8X1 -> connectors:CONN_8X1
- LOGO1: symbol OPEN_HARDWARE_1 -> logo:OPEN_HARDWARE_1
- MOD2: symbol Raspberry_Pi_B2 -> modules:Raspberry_Pi_B2
- R1, R10, R2, R3, R4, R5, R6, R7, R8, R9: symbol R -> standard:R
- SW1: symbol SWITCH -> standard:SWITCH
Connections:
- wire segments 172 -> 197
