File: hw/pi2-base/2relays.sch (KiCad schematic (older format))
At the start: 14 parts, among them Q1 BSS138, Q2 BSS138

Commit message: Fix: Silkscreen jumper description Fix: Relay pinout
Parts:
- REL1, REL2: symbol OMRON_G5LE-1 -> OMRON_G5LE-1-RESCUE-pi2-base
Changed lines of the file:
@@
 EESchema Schematic File Version 2
+LIBS:pi2-base-rescue
 LIBS:connectors
 LIBS:diodes
@@
 LIBS:ics_peripheral
 LIBS:pi2-base-cache
-EELAYER 26 0
+EELAYER 25 0
 EELAYER END
 $Descr A4 11693 8268
@@
 REL2_COM
 $Comp
-L OMRON_G5LE-1 REL2
+L OMRON_G5LE-1-RESCUE-pi2-base REL2
 U 1 1 526EA20C
 P 6725 3800
@@
 $EndComp
 $Comp
-L OMRON_G5LE-1 REL1
+L OMRON_G5LE-1-RESCUE-pi2-base REL1
 U 1 1 526EA068
 P 3925 3800

Commit message: Renamed Rev2 -> RevB Updated 3d footprints Replaced busmodule RevA with RevB symbol
Parts:
- removed REL1, REL2: OMRON_G5LE-1, Relay:omron_G5LE-1, symbol OMRON_G5LE-1-RESCUE-pi2-base
- added REL1, REL2: OMRON_G5LE-1, symbol relays:OMRON_G5LE-1
- D6, D8: symbol D -> standard:D
- D7, D9: symbol LED -> standard:LED
- Q1, Q2: symbol BSS138 -> transistors:BSS138
- R21, R22, R23, R24, R25, R26: symbol R -> standard:R
Connections:
- wire segments 53 -> 66
Changed lines of the file:
@@
-EESchema Schematic File Version 2
-LIBS:pi2-base-rescue
-LIBS:connectors
-LIBS:diodes
-LIBS:ics_regulator
-LIBS:logo
-LIBS:modules
-LIBS:power
-LIBS:relays
-LIBS:standard
-LIBS:transistors
-LIBS:ics_peripheral
+EESchema Schematic File Version 4
 LIBS:pi2-base-cache
-EELAYER 25 0
+EELAYER 26 0
 EELAYER END
 $Descr A4 11693 8268
@@
 Sheet 5 5
 Title "2 Relays"
-Date "2016-12-02"
+Date "2018-09-24"
 Rev "1"
 Comp "KoeWiBa"
@@
 Connection ~ 4050 4700
 Wire Wire Line
-	4150 4700 3975 4700
+	4150 4700 4050 4700
 Wire Wire Line
 	7400 4700 7350 4700
@@
 	7275 3600 7275 3000
 Connection ~ 6475 5300
-Connection ~ 6875 4050
 Connection ~ 6875 4500
 Wire Wire Line
 	6875 4050 6875 4500
 Wire Wire Line
-	7275 4500 6475 4500
+	7275 4500 6875 4500
 Wire Wire Line
 	6475 5300 6475 4900
 Wire Wire Line
-	8075 5300 3675 5300
+	8075 5300 6850 5300
 Wire Wire Line
 	3675 5300 3675 4900
 Wire Wire Line
-	4475 4500 3675 4500
-Wire Wire Line
-	4225 3600 4225 2900
-Wire Wire Line
-	4225 2900 8025 2900
+	4475 4500 4075 4500
+Wire Wire Line
+	4225 2900 7025 2900
 Wire Wire Line
 	4225 4000 4225 4050
 Wire Wire Line
-	4225 4050 3925 4050
-Wire Wire Line
-	3925 4050 3925 3975
-Wire Wire Line
 	4475 4000 4475 4100
 Wire Wire Line
-	3725 3975 3725 4050
-Wire Wire Line
-	3725 4050 3525 4050
-Wire Wire Line
-	3525 4050 3525 3900
-Wire Wire Line
-	3525 3900 3375 3900
-Wire Wire Line
-	3675 3625 3675 3600
-Wire Wire Line
-	3675 3600 3475 3600
-Wire Wire Line
-	3475 3600 3475 3700
-Wire Wire Line
-	3475 3700 3375 3700
-Wire Wire Line
-	3375 3500 3775 3500
-Wire Wire Line
-	3775 3500 3775 3625
-Wire Wire Line
-	3925 3625 3925 3550
-Wire Wire Line
-	3925 3550 4225 3550
-Connection ~ 4225 3550
-Connection ~ 7025 3550
-Wire Wire Line
-	7025 3550 6725 3550
-Wire Wire Line
-	6725 3550 6725 3625
-Wire Wire Line
-	6575 3625 6575 3500
-Wire Wire Line
-	6575 3500 6175 3500
-Wire Wire Line
-	6175 3700 6275 3700
-Wire Wire Line
-	6275 3700 6275 3600
-Wire Wire Line
-	6275 3600 6475 3600
-Wire Wire Line
-	6475 3600 6475 3625
-Wire Wire Line
-	6175 3900 6325 3900
-Wire Wire Line
-	6325 3900 6325 4050
-Wire Wire Line
-	6325 4050 6525 4050
-Wire Wire Line
-	6525 4050 6525 3975
-Wire Wire Line
 	7275 4000 7275 4100
 Wire Wire Line
-	6725 3975 6725 4050
-Wire Wire Line
-	6725 4050 7025 4050
-Wire Wire Line
 	7025 4050 7025 4000
-Wire Wire Line
-	7025 2900 7025 3600
 Connection ~ 7025 2900
 Wire Wire Line
 	4075 4050 4075 4500
 Connection ~ 4075 4500
-Connection ~ 4075 4050
 Wire Wire Line
 	4475 3600 4475 3000
 Wire Wire Line
-	4475 3000 8025 3000
+	4475 3000 7275 3000
 Wire Wire Line
 	6850 4700 6850 4800
 Wire Wire Line
-	6950 4700 6775 4700
+	6950 4700 6850 4700
 Connection ~ 6850 4700
 Wire Wire Line
@@
 LEDVCC
 $Comp
-L BSS138 Q2
+L transistors:BSS138 Q2
 U 1 1 527208FD
 P 6575 4700
@@
 $EndComp
 $Comp
-L R R25
+L standard:R R25
 U 1 1 527208FC
 P 7150 4700
@@
 $EndComp
 $Comp
-L R R22
+L standard:R R22
 U 1 1 527208A4
 P 4350 4700
@@
 $EndComp
 $Comp
-L BSS138 Q1
+L transistors:BSS138 Q1
 U 1 1 5272082F
 P 3775 4700
@@
 Text HLabel 8025 2900 2    50   Input ~ 0
 VCC
-Text HLabel 6175 3700 0    50   UnSpc ~ 0
+Text HLabel 6150 3600 0    50   UnSpc ~ 0
 REL2_NC
-Text HLabel 6175 3500 0    50   UnSpc ~ 0
+Text HLabel 6150 3450 0    50   UnSpc ~ 0
 REL2_NO
-Text HLabel 6175 3900 0    50   UnSpc ~ 0
+Text HLabel 6150 3900 0    50   UnSpc ~ 0
 REL2_COM
 $Comp
-L OMRON_G5LE-1-RESCUE-pi2-base REL2
-U 1 1 526EA20C
-P 6725 3800
-F 0 "REL2" H 6750 3700 50  0000 C CNN
-F 1 "OMRON_G5LE-1" V 7075 3925 50  0000 C CNN
-F 2 "Relay:omron_G5LE-1" H 6725 3800 60  0001 C CNN
-F 3 "" H 6725 3800 60  0001 C CNN
-	1    6725 3800
-	0    -1   -1   0
-$EndComp
-$Comp
-L D D8
+L standard:D D8
 U 1 1 526EA20B
 P 7025 3800
@@
 $EndComp
 $Comp
-L R R24
+L standard:R R24
 U 1 1 526EA20A
 P 6850 5000
@@
 $EndComp
 $Comp
-L R R26
+L standard:R R26
 U 1 1 526EA209
 P 7275 3800
@@
 $EndComp
 $Comp
-L LED D9
+L standard:LED D9
 U 1 1 526EA208
 P 7125 4100
@@
 REL1
 $Comp
-L LED D7
+L standard:LED D7
 U 1 1 526EA113
 P 4325 4100
@@
 $EndComp
 $Comp
-L R R23
+L standard:R R23
 U 1 1 526EA0FD
 P 4475 3800
@@
 $EndComp
 $Comp
-L R R21
+L standard:R R21
 U 1 1 526EA09B
 P 4050 5000
@@
 $EndComp
 $Comp
-L D D6
+L standard:D D6
 U 1 1 526EA082
 P 4225 3800
@@
 	0    -1   -1   0
 $EndComp
-$Comp
-L OMRON_G5LE-1-RESCUE-pi2-base REL1
-U 1 1 526EA068
-P 3925 3800
-F 0 "REL1" H 3950 3700 50  0000 C CNN
-F 1 "OMRON_G5LE-1" V 4275 3925 50  0000 C CNN
-F 2 "Relay:omron_G5LE-1" H 3925 3800 60  0001 C CNN
-F 3 "" H 3925 3800 60  0001 C CNN
-	1    3925 3800
-	0    -1   -1   0
-$EndComp
-Text HLabel 3375 3900 0    50   UnSpc ~ 0
+Text HLabel 3350 3900 0    50   UnSpc ~ 0
 REL1_COM
-Text HLabel 3375 3500 0    50   UnSpc ~ 0
+Text HLabel 3350 3500 0    50   UnSpc ~ 0
 REL1_NO
-Text HLabel 3375 3700 0    50   UnSpc ~ 0
+Text HLabel 3350 3700 0    50   UnSpc ~ 0
 REL1_NC
+Wire Wire Line
+	4050 4700 3975 4700
+Wire Wire Line
+	6850 5300 6475 5300
+Wire Wire Line
+	7275 3000 8025 3000
+Wire Wire Line
+	6475 5300 4050 5300
+Wire Wire Line
+	6875 4050 7025 4050
+Wire Wire Line
+	6875 4500 6475 4500
+Wire Wire Line
+	7025 2900 8025 2900
+Wire Wire Line
+	4075 4500 3675 4500
+Wire Wire Line
+	6850 4700 6775 4700
+Wire Wire Line
+	4050 5300 3675 5300
+$Comp
+L relays:OMRON_G5LE-1 REL2
+U 1 1 5BABA440
+P 6700 3750
+F 0 "REL2" V 7150 4050 50  0000 R CNN
+F 1 "OMRON_G5LE-1" V 7050 4050 50  0000 R CNN
+F 2 "" H 6700 3750 60  0001 C CNN
+F 3 "" H 6700 3750 60  0001 C CNN
+	1    6700 3750
+	0    -1   -1   0
+$EndComp
+$Comp
+L relays:OMRON_G5LE-1 REL1
+U 1 1 5BABA00A
+P 3900 3800
+F 0 "REL1" V 4375 4125 50  0000 R CNN
+F 1 "OMRON_G5LE-1" V 4275 4125 50  0000 R CNN
+F 2 "" H 3900 3800 60  0001 C CNN
+F 3 "" H 3900 3800 60  0001 C CNN
+	1    3900 3800
+	0    -1   -1   0
+$EndComp
+Wire Wire Line
+	4225 2900 4225 3550
+Wire Wire Line
+	4225 4050 4075 4050
+Wire Wire Line
+	3900 4050 3900 4000
+Connection ~ 4075 4050
+Wire Wire Line
+	4075 4050 3900 4050
+Wire Wire Line
+	3900 3600 3900 3550
+Wire Wire Line
+	3900 3550 4225 3550
+Connection ~ 4225 3550
+Wire Wire Line
+	4225 3550 4225 3600
+Wire Wire Line
+	3750 3500 3350 3500
+Wire Wire Line
+	3750 3500 3750 3600
+Wire Wire Line
+	3700 4000 3700 4050
+Wire Wire Line
+	3700 4050 3450 4050
+Wire Wire Line
+	3450 4050 3450 3900
+Wire Wire Line
+	3450 3900 3350 3900
+Wire Wire Line
+	3350 3700 3450 3700
+Wire Wire Line
+	3450 3700 3450 3550
+Wire Wire Line
+	3450 3550 3650 3550
+Wire Wire Line
+	3650 3550 3650 3600
+Wire Wire Line
+	6150 3600 6250 3600
+Wire Wire Line
+	6250 3600 6250 3500
+Wire Wire Line
+	6250 3500 6450 3500
+Wire Wire Line
+	6450 3500 6450 3550
+Wire Wire Line
+	6150 3450 6550 3450
+Wire Wire Line
+	6550 3450 6550 3550
+Wire Wire Line
+	7025 2900 7025 3500
+Wire Wire Line
+	6700 3950 6700 4050
+Wire Wire Line
+	6700 4050 6875 4050
+Connection ~ 6875 4050
+Wire Wire Line
+	6700 3550 6700 3500
+Wire Wire Line
+	6700 3500 7025 3500
+Connection ~ 7025 3500
+Wire Wire Line
+	7025 3500 7025 3600
+Wire Wire Line
+	6150 3900 6250 3900
+Wire Wire Line
+	6250 3900 6250 4000
+Wire Wire Line
+	6250 4000 6500 4000
+Wire Wire Line
+	6500 4000 6500 3950
 $EndSCHEMATC
