File: hw/pi2-base/4inputs.sch (KiCad schematic (older format))
At the start: 12 parts

Commit message: Renamed Rev2 -> RevB Updated 3d footprints Replaced busmodule RevA with RevB symbol
Parts:
- D2, D3, D4, D5: symbol BAT54S -> diodes:BAT54S
- R13, R14, R15, R16, R17, R18, R19, R20: symbol R -> standard:R
Changed lines of the file:
@@
-EESchema Schematic File Version 2
-LIBS:pi2-base-rescue
-LIBS:connectors
-LIBS:diodes
-LIBS:ics_regulator
-LIBS:logo
-LIBS:modules
-LIBS:power
-LIBS:relays
-LIBS:standard
-LIBS:transistors
-LIBS:ics_peripheral
+EESchema Schematic File Version 4
 LIBS:pi2-base-cache
-EELAYER 25 0
+EELAYER 26 0
 EELAYER END
 $Descr A4 11693 8268
@@
 $EndDescr
 $Comp
-L R R13
+L standard:R R13
 U 1 1 52AD89E5
 P 4950 2400
@@
 IN1
 $Comp
-L BAT54S D2
+L diodes:BAT54S D2
 U 1 1 583D5AEB
 P 5450 1800
@@
 	5450 2100 5450 2000
 $Comp
-L R R14
+L standard:R R14
 U 1 1 583D5D3C
 P 4950 3700
@@
 IN2
 $Comp
-L BAT54S D3
+L diodes:BAT54S D3
 U 1 1 583D5D45
 P 5450 3100
@@
 	5450 3400 5450 3300
 $Comp
-L R R15
+L standard:R R15
 U 1 1 583D5EDE
 P 4950 5050
@@
 IN3
 $Comp
-L BAT54S D4
+L diodes:BAT54S D4
 U 1 1 583D5EE7
 P 5450 4450
@@
 	5450 4750 5450 4650
 $Comp
-L R R16
+L standard:R R16
 U 1 1 583D5EF7
 P 4950 6400
@@
 IN4
 $Comp
-L BAT54S D5
+L diodes:BAT54S D5
 U 1 1 583D5F00
 P 5450 5800
@@
 	5450 6100 5450 6000
 $Comp
-L R R18
+L standard:R R18
 U 1 1 584153DB
 P 5150 2850
@@
 $EndComp
 $Comp
-L R R17
+L standard:R R17
 U 1 1 58415503
 P 5150 1550
@@
 	5150 1300 5150 1350
 $Comp
-L R R19
+L standard:R R19
 U 1 1 5841585B
 P 5150 4200
@@
 $EndComp
 $Comp
-L R R20
+L standard:R R20
 U 1 1 584158D3
 P 5150 5550

Commit message: set correct revision to B
Changed lines of the file:
@@
 Title "4 Inputs"
 Date "2016-11-29"
-Rev "1"
+Rev "B"
 Comp "KoeWiBa"
 Comment1 "Baseboard for Raspberry PI 2B"
@@
 $EndComp
 Wire Wire Line
-	5150 1800 5350 1800
+	5150 1800 5250 1800
 Wire Wire Line
 	5250 1800 5250 2400
 Wire Wire Line
-	5150 2400 5550 2400
+	5150 2400 5250 2400
 Connection ~ 5250 2400
 Wire Wire Line
@@
 $EndComp
 Wire Wire Line
-	5150 3100 5350 3100
+	5150 3100 5250 3100
 Wire Wire Line
 	5250 3100 5250 3700
 Wire Wire Line
-	5150 3700 5550 3700
+	5150 3700 5250 3700
 Connection ~ 5250 3700
 Wire Wire Line
@@
 $EndComp
 Wire Wire Line
-	5150 4450 5350 4450
+	5150 4450 5250 4450
 Wire Wire Line
 	5250 4450 5250 5050
 Wire Wire Line
-	5150 5050 5550 5050
+	5150 5050 5250 5050
 Connection ~ 5250 5050
 Wire Wire Line
@@
 $EndComp
 Wire Wire Line
-	5150 5800 5350 5800
+	5150 5800 5250 5800
 Wire Wire Line
 	5250 5800 5250 6400
 Wire Wire Line
-	5150 6400 5550 6400
+	5150 6400 5250 6400
 Connection ~ 5250 6400
 Wire Wire Line
@@
 $EndComp
 Wire Wire Line
-	5150 2600 5550 2600
-Wire Wire Line
-	5150 1300 5550 1300
+	5150 2600 5450 2600
+Wire Wire Line
+	5150 1300 5450 1300
 Connection ~ 5450 1300
 Connection ~ 5450 2600
@@
 	5150 4000 5150 3900
 Wire Wire Line
-	5150 3900 5550 3900
+	5150 3900 5450 3900
 Connection ~ 5450 3900
 Wire Wire Line
-	5150 5250 5550 5250
+	5150 5250 5450 5250
 Wire Wire Line
 	5150 5350 5150 5250
@@
 Text Notes 6100 1550 0    40   ~ 0
 Pulled to ground, a remaining voltage of \n(4700/(4700+56000))*VCC = 0,077 x VCC = 0,38V remains as low voltage.
+Wire Wire Line
+	5250 2400 5550 2400
+Wire Wire Line
+	5250 3700 5550 3700
+Wire Wire Line
+	5250 5050 5550 5050
+Wire Wire Line
+	5250 6400 5550 6400
+Wire Wire Line
+	5450 1300 5550 1300
+Wire Wire Line
+	5450 2600 5550 2600
+Wire Wire Line
+	5250 1800 5350 1800
+Wire Wire Line
+	5250 3100 5350 3100
+Wire Wire Line
+	5250 5800 5350 5800
+Wire Wire Line
+	5250 4450 5350 4450
+Wire Wire Line
+	5450 3900 5550 3900
+Wire Wire Line
+	5450 5250 5550 5250
 $EndSCHEMATC
