File: hw/pi2-base/dcdc.sch (KiCad schematic (older format))
At the start: 8 parts, among them SW2 MAIN, U4 LM2576

Commit message: pi2-base revision 1 (prototypes ordered)
Parts:
- L1: value 220uH -> 100uH
Other:
- note added: "Inductor selected for 24V input voltage and 2A output current"
Changed lines of the file:
@@
 P 6600 3850
 F 0 "L1" H 6500 3750 50  0000 L CNN
-F 1 "220uH" H 6500 3935 50  0000 L CNN
+F 1 "100uH" H 6500 3935 50  0000 L CNN
 F 2 "Inductor:L_PISR" H 6600 3850 60  0001 C CNN
 F 3 "" H 6600 3850 60  0001 C CNN
@@
 Wire Wire Line
 	7500 3350 5250 3350
+Text Notes 5250 3200 0    60   ~ 0
+Inductor selected for 24V input voltage and 2A output current
 $EndSCHEMATC

Commit message: Renamed Rev2 -> RevB Updated 3d footprints Replaced busmodule RevA with RevB symbol
Parts:
- C5, C6: symbol CP -> standard:CP
- D1: symbol SCHOTTKY -> standard:SCHOTTKY
- F2, F3: symbol FUSE -> standard:FUSE
- L1: symbol L -> standard:L
- SW2: symbol SWITCH -> standard:SWITCH
- U4: symbol LM2576 -> ics_regulator:LM2576
Changed lines of the file:
@@
-EESchema Schematic File Version 2
-LIBS:pi2-base-rescue
-LIBS:connectors
-LIBS:diodes
-LIBS:ics_regulator
-LIBS:logo
-LIBS:modules
-LIBS:power
-LIBS:relays
-LIBS:standard
-LIBS:transistors
-LIBS:ics_peripheral
+EESchema Schematic File Version 4
 LIBS:pi2-base-cache
-EELAYER 25 0
+EELAYER 26 0
 EELAYER END
 $Descr A4 11693 8268
@@
 $EndDescr
 Wire Wire Line
-	5250 3350 5250 3900
+	5250 3350 5250 3650
 Wire Wire Line
 	4600 3650 4550 3650
@@
 Connection ~ 5950 4450
 Wire Wire Line
-	6850 4450 5250 4450
-Wire Wire Line
-	6400 3850 6250 3850
+	6850 4450 6325 4450
+Wire Wire Line
+	6400 3850 6325 3850
 Connection ~ 5850 4450
 Connection ~ 5250 3650
@@
 	4150 3750 4150 3800
 Wire Wire Line
-	5450 3650 5000 3650
+	5450 3650 5250 3650
 Wire Wire Line
 	5850 4450 5850 4525
@@
 Connection ~ 6850 3650
 Wire Wire Line
-	6850 3650 6850 3900
+	6850 3650 6850 3850
 Wire Wire Line
 	5250 4450 5250 4200
@@
 	4100 3650 4150 3650
 $Comp
-L LM2576 U4
+L ics_regulator:LM2576 U4
 U 1 1 52AD6D47
 P 5850 3750
@@
 $EndComp
 $Comp
-L SCHOTTKY D1
+L standard:SCHOTTKY D1
 U 1 1 526EC28B
 P 6325 4100
@@
 $EndComp
 $Comp
-L CP C6
+L standard:CP C6
 U 1 1 526EBEBD
 P 6850 4050
@@
 $EndComp
 $Comp
-L L L1
+L standard:L L1
 U 1 1 526EBE7B
 P 6600 3850
@@
 $EndComp
 $Comp
-L GND #PWR024
+L power:GND #PWR024
 U 1 1 526EBE53
 P 5850 4525
@@
 $EndComp
 $Comp
-L CP C5
+L standard:CP C5
 U 1 1 526EBE2E
 P 5250 4050
@@
 $EndComp
 $Comp
-L SWITCH SW2
+L standard:SWITCH SW2
 U 1 1 526EA5A3
 P 4100 3750
@@
 $EndComp
 $Comp
-L GND #PWR025
+L power:GND #PWR025
 U 1 1 526EA53B
 P 4150 3800
@@
 $EndComp
 $Comp
-L FUSE F3
+L standard:FUSE F3
 U 1 1 583C6A9F
 P 7150 3650
@@
 $EndComp
 $Comp
-L FUSE F2
+L standard:FUSE F2
 U 1 1 583C71B1
 P 4800 3650
@@
 GND
 Wire Wire Line
-	6250 3650 6950 3650
+	6250 3650 6850 3650
 Wire Wire Line
 	7350 3650 7500 3650
@@
 Text Notes 5250 3200 0    60   ~ 0
 Inductor selected for 24V input voltage and 2A output current
+Wire Wire Line
+	5950 4450 5850 4450
+Wire Wire Line
+	5850 4450 5750 4450
+Wire Wire Line
+	5250 3650 5250 3900
+Wire Wire Line
+	5250 3650 5000 3650
+Wire Wire Line
+	5750 4450 5250 4450
+Wire Wire Line
+	6850 3850 6850 3900
+Wire Wire Line
+	6850 3650 6950 3650
+Wire Wire Line
+	6325 4450 5950 4450
+Wire Wire Line
+	6325 3850 6250 3850
 $EndSCHEMATC
