File: hw/pi2-base/rtc.sch (KiCad schematic (older format))
At the start: 10 parts, among them U1 PCA9517, U2 DS1307, U3 32.768kHz

Commit message: Renamed Rev2 -> RevB Updated 3d footprints Replaced busmodule RevA with RevB symbol
Parts:
- BATT1: symbol BATT -> standard:BATT
- C1, C2, C3, C4: symbol C -> standard:C
- R11, R12: symbol R -> standard:R
- U1: symbol PCA9517 -> ics_peripheral:PCA9517
- U2: symbol DS1307 -> ics_peripheral:DS1307
- U3: symbol CRYSTAL -> standard:CRYSTAL
Changed lines of the file:
@@
-EESchema Schematic File Version 2
-LIBS:pi2-base-rescue
-LIBS:connectors
-LIBS:diodes
-LIBS:ics_regulator
-LIBS:logo
-LIBS:modules
-LIBS:power
-LIBS:relays
-LIBS:standard
-LIBS:transistors
-LIBS:ics_peripheral
+EESchema Schematic File Version 4
 LIBS:pi2-base-cache
-EELAYER 25 0
+EELAYER 26 0
 EELAYER END
 $Descr A4 11693 8268
@@
 SCL
 $Comp
-L C C1
+L standard:C C1
 U 1 1 527FA60F
 P 5550 4350
@@
 $EndComp
 $Comp
-L BATT BATT1
+L standard:BATT BATT1
 U 1 1 527FA283
 P 7900 4200
@@
 $EndComp
 $Comp
-L C C2
+L standard:C C2
 U 1 1 527FA128
 P 6300 4200
@@
 $EndComp
 $Comp
-L C C4
+L standard:C C4
 U 1 1 527FA124
 P 8250 3900
@@
 $EndComp
 $Comp
-L C C3
+L standard:C C3
 U 1 1 527FA121
 P 8250 3700
@@
 $EndComp
 $Comp
-L CRYSTAL U3
+L standard:CRYSTAL U3
 U 1 1 527FA110
 P 7700 3800
@@
 $EndComp
 $Comp
-L DS1307 U2
+L ics_peripheral:DS1307 U2
 U 1 1 527F9F98
 P 7050 3900
@@
 $EndComp
 $Comp
-L PCA9517 U1
+L ics_peripheral:PCA9517 U1
 U 1 1 527F9F8E
 P 4900 4000
@@
 	4000 4100 3900 4100
 $Comp
-L R R11
+L standard:R R11
 U 1 1 583C425A
 P 5800 3650
@@
 $EndComp
 $Comp
-L R R12
+L standard:R R12
 U 1 1 583C4352
 P 6050 3650

Commit message: set correct revision to B
Changed lines of the file:
@@
 Title "RTC"
 Date "2016-11-28"
-Rev "1"
+Rev "B"
 Comp "KoeWiBa"
 Comment1 "Baseboard for Raspberry PI 2"
@@
 	4000 3950 4350 3950
 Wire Wire Line
-	5450 3950 6500 3950
-Wire Wire Line
-	5450 4050 6500 4050
+	5450 3950 5800 3950
+Wire Wire Line
+	5450 4050 6050 4050
 Connection ~ 5550 3850
 Wire Wire Line
@@
 	7700 3850 7700 3900
 Wire Wire Line
-	7700 3900 8150 3900
+	7700 3900 8050 3900
 Wire Wire Line
 	7700 3750 7600 3750
@@
 	8150 3700 7700 3700
 Wire Wire Line
-	7700 3700 7700 3800
+	7700 3700 7700 3750
 Connection ~ 7700 3750
 Wire Wire Line
@@
 	6300 3750 6500 3750
 Wire Wire Line
-	8400 3700 8400 4350
-Wire Wire Line
-	8400 4350 6300 4350
+	8400 3700 8400 3900
+Wire Wire Line
+	8400 4350 7900 4350
 Connection ~ 7900 4350
 Wire Wire Line
@@
 	7900 4300 7900 4350
 Wire Wire Line
-	5550 3400 5550 4250
+	5550 3400 5550 3850
 Wire Wire Line
 	4000 4050 4350 4050
 Wire Wire Line
-	6300 3250 6300 4100
+	6300 3250 6300 3400
 Connection ~ 6300 3750
 Text Label 4300 4050 2    40   ~ 0
@@
 	4250 4150 4250 4650
 Wire Wire Line
-	5550 4450 5550 4750
+	5550 4450 5550 4650
 Text HLabel 3900 3900 0    50   Input ~ 0
 SCL_3V3
@@
 	5800 3450 5800 3400
 Wire Wire Line
-	5550 3400 6300 3400
+	5550 3400 5800 3400
 Wire Wire Line
 	6050 3450 6050 3400
@@
 	4250 3850 4250 3200
 Wire Wire Line
-	4250 4650 7300 4650
+	4250 4650 5550 4650
 Connection ~ 5550 4650
 Text HLabel 5550 4750 3    50   Input ~ 0
 GND
+Wire Wire Line
+	5550 3850 5550 4250
+Wire Wire Line
+	7300 4350 6300 4350
+Wire Wire Line
+	7700 4350 7300 4350
+Wire Wire Line
+	8400 3900 8400 4350
+Wire Wire Line
+	8050 3900 8150 3900
+Wire Wire Line
+	7700 3750 7700 3800
+Wire Wire Line
+	7900 4350 7700 4350
+Wire Wire Line
+	6300 3750 6300 4100
+Wire Wire Line
+	6050 3400 6300 3400
+Wire Wire Line
+	6300 3400 6300 3750
+Wire Wire Line
+	5800 3950 6500 3950
+Wire Wire Line
+	6050 4050 6500 4050
+Wire Wire Line
+	5800 3400 6050 3400
+Wire Wire Line
+	5550 4650 5550 4750
+Wire Wire Line
+	5550 4650 7300 4650
 $EndSCHEMATC
