File: hw/bus-module_atmega328/bus-module_atmega328.kicad_pcb (KiCad board)
At the start: 2 copper layers, 35 x 48 mm, 31 parts, among them J1 CONN_10X2, J2 CONN_7X2, J3 CONN-ISP-6, J5 CONN_1, J6 CONN_1, J7 CONN_1, J8 CONN_1, U1 ATMEGA328-TQFP32, U2 7,3728MHz, U3 25LC256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

Commit message: Start of development of Rev. B: - integrated fuse for 24V supply. - new footprint SOT143 for TVS-Diode. - replaced TVS-Diode footprint by SOT143. - added revision text on copper layer.
Parts:
- added F1: FUSE, Resistor:R_1812, F.Cu at (83.4, 104.2)
- D2: footprint Housings_SOT:SOT143R_Diode_Reverse -> Diode_SMD:SOT143
- moved D2 0.52 mm to (83.1, 97.3), turned to 90 degrees
Connections:
- J5 pad 1: +24V -> Net-(F1-Pad2)
Routing:
- net /B: track 21.4 -> 12.9 mm, vias 1 -> 0
- net Net-(F1-Pad2): track 0.00 -> 3.89 mm
- net +24V: track 6.65 -> 10.5 mm
- net GND: track 44.2 -> 41.6 mm
- net /A: track 17.4 -> 17.7 mm, vias 1 -> 0
Other:
- board text added: "Rev. B"

Commit message: SPI resistors changed from 1k to 100
Parts:
- R2, R3, R4: value 1k -> 100
Changed lines of the file:
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@@
-(kicad_pcb (version 4) (host pcbnew "(2015-09-05 BZR 6159)-product")
+(kicad_pcb (version 20170123) (host pcbnew no-vcs-found-7600~57~ubuntu14.04.1)
   (general
     (links 93)
     (no_connects 0)
-    (area 52.678572 64.65 152.455 131.450001)
+    (area 79.949999 75.947965 115.054227 124.050001)
     (thickness 1.6)
     (drawings 40)
@@
       (hpglpenspeed 20)
       (hpglpendiameter 15)
-      (hpglpenoverlay 2)
       (psnegative false)
       (psa4output false)
@@
     (at 99 107.01 270)
     (attr smd)
-    (fp_text reference R2 (at 2.3 -0.175 360) (layer F.SilkS)
-      (effects (font (size 0.6096 0.6096) (thickness 0.1016)))
-    )
-    (fp_text value 1k (at 0 0 270) (layer F.SilkS) hide
+    (fp_text reference R2 (at 2.3 -0.175) (layer F.SilkS)
+      (effects (font (size 0.6096 0.6096) (thickness 0.1016)))
+    )
+    (fp_text value 100 (at 0 0 270) (layer F.SilkS) hide
       (effects (font (size 0.6096 0.6096) (thickness 0.1016)))
     )
@@
     (at 101.25 107.01 270)
     (attr smd)
-    (fp_text reference R4 (at 2.3 -0.025 360) (layer F.SilkS)
-      (effects (font (size 0.6096 0.6096) (thickness 0.1016)))
-    )
-    (fp_text value 1k (at 0 0 270) (layer F.SilkS) hide
+    (fp_text reference R4 (at 2.3 -0.025) (layer F.SilkS)
+      (effects (font (size 0.6096 0.6096) (thickness 0.1016)))
+    )
+    (fp_text value 100 (at 0 0 270) (layer F.SilkS) hide
       (effects (font (size 0.6096 0.6096) (thickness 0.1016)))
     )
@@
   (module Connector_Header:HEADER_3x2 (layer B.Cu)
     (at 112.25 112.21 270)
-    (fp_text reference J3 (at -2.41 1.25 360) (layer B.SilkS)
+    (fp_text reference J3 (at -2.41 1.25) (layer B.SilkS)
       (effects (font (size 1 1) (thickness 0.15)) (justify mirror))
     )
@@
     (at 106.863 107.032 270)
     (attr smd)
-    (fp_text reference C6 (at 2.5 -0.05 360) (layer F.SilkS)
+    (fp_text reference C6 (at 2.5 -0.05) (layer F.SilkS)
       (effects (font (size 0.6096 0.6096) (thickness 0.1016)))
     )
@@
     (at 96.75 106.9625 270)
     (attr smd)
-    (fp_text reference R3 (at -2.3525 0 540) (layer F.SilkS)
-      (effects (font (size 0.6096 0.6096) (thickness 0.1016)))
-    )
-    (fp_text value 1k (at 0 0 270) (layer F.SilkS) hide
+    (fp_text reference R3 (at -2.3525 0 180) (layer F.SilkS)
+      (effects (font (size 0.6096 0.6096) (thickness 0.1016)))
+    )
+    (fp_text value 100 (at 0 0 270) (layer F.SilkS) hide
       (effects (font (size 0.6096 0.6096) (thickness 0.1016)))
     )
@@
     (at 106.9525 88 180)
     (attr smd)
-    (fp_text reference R6 (at -3.0225 -0.01 360) (layer F.SilkS)
+    (fp_text reference R6 (at -3.0225 -0.01) (layer F.SilkS)
       (effects (font (size 0.6096 0.6096) (thickness 0.1016)))
     )
@@
     (tags "CMS SOJ")
     (attr smd)
-    (fp_text reference U3 (at -3.5 0 360) (layer F.SilkS)
+    (fp_text reference U3 (at -3.5 0) (layer F.SilkS)
       (effects (font (size 1 1) (thickness 0.15)))
     )
@@
     (tags "CMS SOJ")
     (attr smd)
-    (fp_text reference U4 (at -3.95 -2.6 360) (layer B.SilkS)
+    (fp_text reference U4 (at -3.95 -2.6) (layer B.SilkS)
       (effects (font (size 1 1) (thickness 0.15)) (justify mirror))
     )
@@
       (effects (font (size 0.8 0.8) (thickness 0.15)))
     )
-    (fp_text value FUSE (at 0 0.0508 360) (layer F.Fab)
+    (fp_text value FUSE (at 0 0.0508) (layer F.Fab)
       (effects (font (size 0.8 0.8) (thickness 0.15)))
     )
