File: hw/bus-module_atmega328/bus-module_atmega328.sch (KiCad schematic (older format))
At the start: 31 parts, among them J1 CONN_10X2, J2 CONN_7X2, J3 CONN-ISP-6, J5 CONN_1, J6 CONN_1, J7 CONN_1, J8 CONN_1, U1 ATMEGA328-TQFP32, U2 7,3728MHz, U3 25LC256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

Commit message: Start of development of Rev. B: - integrated fuse for 24V supply. - new footprint SOT143 for TVS-Diode. - replaced TVS-Diode footprint by SOT143. - added revision text on copper layer.
Parts:
- added F1: FUSE, Resistor:R_1812, symbol FUSE
- D2: footprint Housings_SOT:SOT143R_Diode_Reverse -> Diode_SMD:SOT143
Connections:
- net +24V: now also F1.1; no longer J5.1
- new net: F1.2, J5.1
Changed lines of the file:
@@
 EESchema Schematic File Version 2
-LIBS:bus-module_atmega328-rescue
 LIBS:connectors
-LIBS:display
-LIBS:encoder
-LIBS:ics_40xx
+LIBS:diodes
 LIBS:ics_controller_atmel
 LIBS:ics_misc
-LIBS:ics_opamp
-LIBS:ics_opto
 LIBS:ics_peripheral
 LIBS:ics_regulator
 LIBS:logo
 LIBS:power
-LIBS:relays
-LIBS:sensors
 LIBS:standard
-LIBS:transformer
-LIBS:transistors
-LIBS:diodes
 LIBS:bus-module_atmega328-cache
 EELAYER 25 0
@@
 L +24V #PWR03
 U 1 1 559D77F1
-P 9950 2400
-F 0 "#PWR03" H 9950 2600 50  0001 C CNN
-F 1 "+24V" H 9950 2510 50  0000 C CNN
-F 2 "" H 9950 2400 60  0000 C CNN
-F 3 "" H 9950 2400 60  0000 C CNN
-	1    9950 2400
+P 9350 2400
+F 0 "#PWR03" H 9350 2600 50  0001 C CNN
+F 1 "+24V" H 9350 2510 50  0000 C CNN
+F 2 "" H 9350 2400 60  0000 C CNN
+F 3 "" H 9350 2400 60  0000 C CNN
+	1    9350 2400
 	1    0    0    -1
 $EndComp
@@
 	6750 3100 6850 3000
 Wire Bus Line
-	6750 5800 6750 2750
+	6750 2750 6750 5800
 Wire Wire Line
 	8350 2900 10050 2900
@@
 	4300 5700 4700 5700
 Wire Bus Line
-	5400 5600 5400 5800
+	5400 5800 5400 5600
 Text Label 4300 6700 0    40   ~ 0
 /CSEEP
@@
 	5900 6800 5750 6800
 Wire Wire Line
-	5900 6200 5900 6150
-Wire Wire Line
-	5900 6150 4550 6150
+	5900 6150 5900 6200
+Wire Wire Line
+	4550 6150 5900 6150
 Wire Wire Line
 	4550 6150 4550 6200
@@
 	1    0    0    -1
 $EndComp
-Wire Wire Line
-	9950 2400 9950 2500
 Wire Wire Line
 	10050 3100 9950 3100
@@
 	5450 2100 5450 2350
 Wire Wire Line
-	6650 2750 6150 2750
+	6150 2750 6650 2750
 Wire Wire Line
 	6250 2150 6250 2750
@@
 	1500 4500 1600 4400
 Wire Bus Line
-	1500 5800 1500 2800
+	1500 2800 1500 5800
 Wire Wire Line
 	1600 3900 1950 3900
@@
 $EndComp
 Wire Bus Line
-	5400 5800 1500 5800
+	1500 5800 5400 5800
 $Comp
 L SEMTECH_SR05 D2
@@
 F 0 "D2" H 9125 3450 50  0000 C CNN
 F 1 "SEMTECH SR05" H 9050 4050 50  0000 C CNN
-F 2 "Housings_SOT:SOT143R_Diode_Reverse" H 9050 3700 60  0001 C CNN
+F 2 "Diode_SMD:SOT143" H 9050 3700 60  0001 C CNN
 F 3 "" H 9050 3700 60  0000 C CNN
 	1    9050 3700
@@
 $EndComp
 Wire Wire Line
-	9950 2500 10050 2500
-Wire Wire Line
 	8350 3000 8100 3000
 Wire Wire Line
 	9550 4200 9550 4100
 Wire Wire Line
-	6750 1450 4950 1450
+	4950 1450 6750 1450
 Wire Wire Line
 	4950 1450 4950 1700
@@
 Text Label 9200 2900 0    40   ~ 0
 B
+$Comp
+L FUSE F1
+U 1 1 56648405
+P 9750 2500
+F 0 "F1" H 9750 2600 50  0000 C CNN
+F 1 "FUSE" H 9750 2400 50  0000 C CNN
+F 2 "Resistor:R_1812" H 9750 2500 60  0001 C CNN
+F 3 "" H 9750 2500 60  0000 C CNN
+	1    9750 2500
+	1    0    0    -1
+$EndComp
+Wire Wire Line
+	9350 2400 9350 2500
+Wire Wire Line
+	9350 2500 9550 2500
+Wire Wire Line
+	9950 2500 10050 2500
 $EndSCHEMATC

Commit message: SPI resistors changed from 1k to 100
Parts:
- R2, R3, R4: value 1k -> 100
Changed lines of the file:
@@
 LIBS:standard
 LIBS:bus-module_atmega328-cache
-EELAYER 25 0
+EELAYER 26 0
 EELAYER END
 $Descr A4 11693 8268
@@
 Sheet 1 1
 Title "bus-module_atmega328"
-Date "2015-10-19"
+Date "2017-02-10"
 Rev "1"
 Comp "KoeWiBa"
@@
 P 4900 5700
 F 0 "R4" H 4100 5700 50  0000 C CNN
-F 1 "1k" H 4900 5700 50  0000 C CNN
+F 1 "100" H 4900 5700 50  0000 C CNN
 F 2 "Housings_SOIC:SM0805" H 4900 5700 60  0001 C CNN
 F 3 "" H 4900 5700 60  0000 C CNN
@@
 P 4900 5600
 F 0 "R3" H 4100 5600 50  0000 C CNN
-F 1 "1k" H 4900 5600 50  0000 C CNN
+F 1 "100" H 4900 5600 50  0000 C CNN
 F 2 "Housings_SOIC:SM0805" H 4900 5600 60  0001 C CNN
 F 3 "" H 4900 5600 60  0000 C CNN
@@
 P 4900 5500
 F 0 "R2" H 4100 5500 50  0000 C CNN
-F 1 "1k" H 4900 5500 50  0000 C CNN
+F 1 "100" H 4900 5500 50  0000 C CNN
 F 2 "Housings_SOIC:SM0805" H 4900 5500 60  0001 C CNN
 F 3 "" H 4900 5500 60  0000 C CNN
