File: hw/bus-module_atmega328/bus-module_atmega328.sch (KiCad schematic (older format))
At the start: 31 parts, among them J1 CONN_10X2, J2 CONN_7X2, J3 CONN-ISP-6, J5 CONN_1, J6 CONN_1, J7 CONN_1, J8 CONN_1, U1 ATMEGA328-TQFP32, U2 7,3728MHz, U3 25LC256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

Commit message: bus-module_atmega328 update to rev B
Parts:
- added F1: FUSE, Resistor:R_1812, symbol bus-module_atmega328-rescue:FUSE
- C1, C2, C3, C5, C6, C7, C8: symbol C -> standard:C
- C9: symbol CP -> standard:CP
- D1: symbol D -> standard:D
- D2: footprint Housings_SOT:SOT143R_Diode_Reverse -> Diode_SMD:SOT143; symbol SEMTECH_SR05 -> diodes:SEMTECH_SR05
- H1: symbol HOLE -> standard:HOLE
- J1: symbol CONN_10X2 -> connectors:CONN_10X2
- J2: symbol CONN_7X2 -> connectors:CONN_7X2
- J3: symbol CONN-ISP-6 -> connectors:CONN-ISP-6
- J5, J6, J7, J8: symbol CONN_1 -> connectors:CONN_1
- L1: symbol L -> standard:L
- LOGO1: symbol OPEN_HARDWARE_1 -> logo:OPEN_HARDWARE_1
- R1, R2, R3, R4, R5, R6: symbol R -> standard:R
- U1: symbol ATMEGA88-TQFP32 -> ics_controller_atmel:ATMEGA88-TQFP32
- U2: symbol CRYSTAL -> standard:CRYSTAL
- U3: symbol 25LCXXX -> ics_peripheral:25LCXXX
- U4: symbol MAX487 -> ics_misc:MAX487
- U5: symbol AM1S-2403 -> ics_regulator:AM1S-2403
Connections:
- net +24V: now also J1.3, J1.4, F1.2; no longer U5.2 (VIN+)
- net VCC: no longer J1.3, J1.4
- new net: F1.1, U5.2 (VIN+)
