File: hw/bus-module_attiny1634/bus-module_attiny1634.kicad_pcb (KiCad board)
At the start: 2 copper layers, 27.3 x 48 mm, 36 parts, among them J1 CONN_5X2, J2 CONN_5X2, J3 CONN-ISP-6, J4 CONN_1, J5 CONN_1, J6 CONN_1, J7 CONN_1, U1 7,3728MHz, U2 25LCXXX, U3 ATtiny1634-SOIC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

Commit message: Start of development of Rev. B: - integrated fuse for 24V supply. - new footprint SOT143 for TVS-Diode. - replaced TVS-Diode footprint by SOT143. - added revision text on copper layer.
Parts:
- added F1: FUSE, Resistor:R_1812, F.Cu at (82.9, 104.5)
- D2: footprint Housings_SOT:SOT143R_Diode_Reverse -> Diode_SMD:SOT143
- moved D2 1.00 mm to (83.3, 97.3), turned to 90 degrees
Connections:
- J4 pad 1: +24V -> Net-(F1-Pad2)
Routing:
- net +5V: track 28.4 -> 46.4 mm, vias 3 -> 4
- net /B: track 25.2 -> 18.6 mm, vias 1 -> 0
- net GND: track 15.8 -> 22.2 mm, vias 5 -> 4
- net /A: track 31.5 -> 25.6 mm, vias 1 -> 0
- net +24V: track 20.6 -> 25.3 mm
- net Net-(F1-Pad2): track 0.00 -> 4.57 mm
- net //RESET: track 53.9 -> 55.0 mm
Other:
- board text added: "Rev. B"

Commit message: SPI resistors changed from 1k to 100
Parts:
- R2, R3, R4: value 1k -> 100
Changed lines of the file:
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@@
-(kicad_pcb (version 4) (host pcbnew "(2015-09-05 BZR 6159)-product")
+(kicad_pcb (version 20170123) (host pcbnew no-vcs-found-7600~57~ubuntu14.04.1)
   (general
     (links 78)
     (no_connects 0)
-    (area 52.678572 66.17 119.506 125.354001)
+    (area 79.949999 75.949999 107.365001 124.050001)
     (thickness 1.6)
     (drawings 41)
@@
       (hpglpenspeed 20)
       (hpglpendiameter 15)
-      (hpglpenoverlay 2)
       (psnegative false)
       (psa4output false)
@@
   (module Connector_Header:HEADER_3x2 (layer B.Cu)
     (at 92.448 83.32 180)
-    (fp_text reference J3 (at 2.54 4.826 360) (layer B.SilkS)
+    (fp_text reference J3 (at 2.54 4.826) (layer B.SilkS)
       (effects (font (size 1 1) (thickness 0.15)) (justify mirror))
     )
@@
     (at 96.512 89.416 270)
     (attr smd)
-    (fp_text reference C1 (at -2.286 3.556 360) (layer B.SilkS)
+    (fp_text reference C1 (at -2.286 3.556) (layer B.SilkS)
       (effects (font (size 0.6096 0.6096) (thickness 0.1016)) (justify mirror))
     )
@@
     (at 92.448 105.164 270)
     (attr smd)
-    (fp_text reference C2 (at 0 1.778 360) (layer F.SilkS)
+    (fp_text reference C2 (at 0 1.778) (layer F.SilkS)
       (effects (font (size 0.6096 0.6096) (thickness 0.1016)))
     )
@@
     (at 104.64 89.416 270)
     (attr smd)
-    (fp_text reference R1 (at -2.286 5.588 360) (layer B.SilkS)
+    (fp_text reference R1 (at -2.286 5.588) (layer B.SilkS)
       (effects (font (size 0.6096 0.6096) (thickness 0.1016)) (justify mirror))
     )
@@
     (at 105.91 102.116 270)
     (attr smd)
-    (fp_text reference R2 (at 2.54 0 360) (layer F.SilkS)
-      (effects (font (size 0.6096 0.6096) (thickness 0.1016)))
-    )
-    (fp_text value 1k (at 0.127 1.524 270) (layer F.SilkS) hide
+    (fp_text reference R2 (at 2.54 0) (layer F.SilkS)
+      (effects (font (size 0.6096 0.6096) (thickness 0.1016)))
+    )
+    (fp_text value 100 (at 0.127 1.524 270) (layer F.SilkS) hide
       (effects (font (size 0.6096 0.6096) (thickness 0.1016)))
     )
@@
     (at 103.878 102.116 270)
     (attr smd)
-    (fp_text reference R3 (at 2.54 0 360) (layer F.SilkS)
-      (effects (font (size 0.6096 0.6096) (thickness 0.1016)))
-    )
-    (fp_text value 1k (at 0.127 1.524 270) (layer F.SilkS) hide
+    (fp_text reference R3 (at 2.54 0) (layer F.SilkS)
+      (effects (font (size 0.6096 0.6096) (thickness 0.1016)))
+    )
+    (fp_text value 100 (at 0.127 1.524 270) (layer F.SilkS) hide
       (effects (font (size 0.6096 0.6096) (thickness 0.1016)))
     )
@@
     (at 101.338 102.116 270)
     (attr smd)
-    (fp_text reference R4 (at 2.54 0 360) (layer F.SilkS)
-      (effects (font (size 0.6096 0.6096) (thickness 0.1016)))
-    )
-    (fp_text value 1k (at 0.127 1.524 270) (layer F.SilkS) hide
+    (fp_text reference R4 (at 2.54 0) (layer F.SilkS)
+      (effects (font (size 0.6096 0.6096) (thickness 0.1016)))
+    )
+    (fp_text value 100 (at 0.127 1.524 270) (layer F.SilkS) hide
       (effects (font (size 0.6096 0.6096) (thickness 0.1016)))
     )
@@
     (at 98.544 89.416 270)
     (attr smd)
-    (fp_text reference R5 (at -2.286 4.064 360) (layer B.SilkS)
+    (fp_text reference R5 (at -2.286 4.064) (layer B.SilkS)
       (effects (font (size 0.6096 0.6096) (thickness 0.1016)) (justify mirror))
     )
@@
     (at 102.1 89.416 270)
     (attr smd)
-    (fp_text reference R6 (at -2.286 4.572 360) (layer B.SilkS)
+    (fp_text reference R6 (at -2.286 4.572) (layer B.SilkS)
       (effects (font (size 0.6096 0.6096) (thickness 0.1016)) (justify mirror))
     )
@@
     (at 96.004 102.116 270)
     (attr smd)
-    (fp_text reference C4 (at 0 -1.778 360) (layer B.SilkS)
+    (fp_text reference C4 (at 0 -1.778) (layer B.SilkS)
       (effects (font (size 0.6096 0.6096) (thickness 0.1016)) (justify mirror))
     )
@@
   (module Crystal:HC49-SMD (layer F.Cu)
     (at 96.512 107.01058 270)
-    (fp_text reference U1 (at 5.51942 3.81 360) (layer F.SilkS)
+    (fp_text reference U1 (at 5.51942 3.81) (layer F.SilkS)
       (effects (font (size 1.016 1.016) (thickness 0.15)))
     )
@@
       (effects (font (size 0.8 0.8) (thickness 0.15)))
     )
-    (fp_text value FUSE (at 0 0.0508 360) (layer F.Fab)
+    (fp_text value FUSE (at 0 0.0508) (layer F.Fab)
       (effects (font (size 0.8 0.8) (thickness 0.15)))
     )
