File: hw/bus-module_attiny1634/bus-module_attiny1634.sch (KiCad schematic (older format))
At the start: 30 parts, among them J1 CONN_5X2, J2 CONN_5X2, J3 CONN-ISP-6, J4 CONN_1, J5 CONN_1, J6 CONN_1, J7 CONN_1, U1 7,3728MHz, U2 25LCXXX, U3 ATtiny1634-SOIC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

Commit message: initial revision of bus-module_attiny1634 revB. not checked yet
Parts:
- added F1: FUSE, Resistor:R_1812, symbol FUSE
- D2: footprint Housings_SOT:SOT143R_Diode_Reverse -> Diode_SMD:SOT143
Connections:
- net +24V: now also J1.3, J1.4, F1.2; no longer R7.1, U5.2 (VIN+)
- net +5V: no longer J1.3, J1.4
- new net: F1.1, R7.1, U5.2 (VIN+)
Other:
- moved on the sheet: J4, J5, J6, J7, R7
Changed lines of the file:
@@
 EESchema Schematic File Version 2
-LIBS:connectors
-LIBS:diodes
-LIBS:ics_controller_atmel
-LIBS:ics_misc
-LIBS:ics_peripheral
-LIBS:ics_regulator
-LIBS:logo
-LIBS:power
-LIBS:standard
 LIBS:bus-module_attiny1634-cache
 EELAYER 25 0
@@
 Sheet 1 1
 Title "bus-module_attiny1634"
-Date "2015-10-28"
-Rev "1"
+Date "2015-12-06"
+Rev "2"
 Comp "KoeWiBa"
 Comment1 ""
@@
 L CONN_1 J4
 U 1 1 559D5A6B
-P 9900 2500
-F 0 "J4" H 9900 2575 50  0000 C CNN
-F 1 "CONN_1" H 9900 2425 25  0000 C CNN
-F 2 "Connector_Miscelleaneus:WAGO243" H 9900 2500 60  0001 C CNN
-F 3 "" H 9900 2500 60  0000 C CNN
-	1    9900 2500
+P 10400 2500
+F 0 "J4" H 10400 2575 50  0000 C CNN
+F 1 "CONN_1" H 10400 2425 25  0000 C CNN
+F 2 "Connector_Miscelleaneus:WAGO243" H 10400 2500 60  0001 C CNN
+F 3 "" H 10400 2500 60  0000 C CNN
+	1    10400 2500
 	1    0    0    -1
 $EndComp
@@
 L CONN_1 J5
 U 1 1 559D5ACC
-P 9900 2700
-F 0 "J5" H 9900 2775 50  0000 C CNN
-F 1 "CONN_1" H 9900 2625 25  0000 C CNN
-F 2 "Connector_Miscelleaneus:WAGO243" H 9900 2700 60  0001 C CNN
-F 3 "" H 9900 2700 60  0000 C CNN
-	1    9900 2700
+P 10400 2700
+F 0 "J5" H 10400 2775 50  0000 C CNN
+F 1 "CONN_1" H 10400 2625 25  0000 C CNN
+F 2 "Connector_Miscelleaneus:WAGO243" H 10400 2700 60  0001 C CNN
+F 3 "" H 10400 2700 60  0000 C CNN
+	1    10400 2700
 	1    0    0    -1
 $EndComp
@@
 L CONN_1 J6
 U 1 1 559D5B5B
-P 9900 2900
-F 0 "J6" H 9900 2975 50  0000 C CNN
-F 1 "CONN_1" H 9900 2825 25  0000 C CNN
-F 2 "Connector_Miscelleaneus:WAGO243" H 9900 2900 60  0001 C CNN
-F 3 "" H 9900 2900 60  0000 C CNN
-	1    9900 2900
+P 10400 2900
+F 0 "J6" H 10400 2975 50  0000 C CNN
+F 1 "CONN_1" H 10400 2825 25  0000 C CNN
+F 2 "Connector_Miscelleaneus:WAGO243" H 10400 2900 60  0001 C CNN
+F 3 "" H 10400 2900 60  0000 C CNN
+	1    10400 2900
 	1    0    0    -1
 $EndComp
@@
 L CONN_1 J7
 U 1 1 559D5B94
-P 9900 3100
-F 0 "J7" H 9900 3175 50  0000 C CNN
-F 1 "CONN_1" H 9900 3025 25  0000 C CNN
-F 2 "Connector_Miscelleaneus:WAGO243" H 9900 3100 60  0001 C CNN
-F 3 "" H 9900 3100 60  0000 C CNN
-	1    9900 3100
+P 10400 3100
+F 0 "J7" H 10400 3175 50  0000 C CNN
+F 1 "CONN_1" H 10400 3025 25  0000 C CNN
+F 2 "Connector_Miscelleaneus:WAGO243" H 10400 3100 60  0001 C CNN
+F 3 "" H 10400 3100 60  0000 C CNN
+	1    10400 3100
 	1    0    0    -1
 $EndComp
@@
 L +24V #PWR03
 U 1 1 559D77F1
-P 9700 2400
-F 0 "#PWR03" H 9700 2600 50  0001 C CNN
-F 1 "+24V" H 9700 2510 50  0000 C CNN
-F 2 "" H 9700 2400 60  0000 C CNN
-F 3 "" H 9700 2400 60  0000 C CNN
-	1    9700 2400
+P 10100 2400
+F 0 "#PWR03" H 10100 2600 50  0001 C CNN
+F 1 "+24V" H 10100 2510 50  0000 C CNN
+F 2 "" H 10100 2400 60  0000 C CNN
+F 3 "" H 10100 2400 60  0000 C CNN
+	1    10100 2400
 	1    0    0    -1
 $EndComp
@@
 L +24V #PWR010
 U 1 1 55A0FF09
-P 8650 1100
-F 0 "#PWR010" H 8650 1300 50  0001 C CNN
-F 1 "+24V" H 8650 1210 50  0000 C CNN
-F 2 "" H 8650 1100 60  0000 C CNN
-F 3 "" H 8650 1100 60  0000 C CNN
-	1    8650 1100
+P 9600 1100
+F 0 "#PWR010" H 9600 1300 50  0001 C CNN
+F 1 "+24V" H 9600 1210 50  0000 C CNN
+F 2 "" H 9600 1100 60  0000 C CNN
+F 3 "" H 9600 1100 60  0000 C CNN
+	1    9600 1100
 	1    0    0    -1
 $EndComp
@@
 L GND #PWR011
 U 1 1 55A10203
-P 8650 1500
-F 0 "#PWR011" H 8650 1300 50  0001 C CNN
-F 1 "GND" H 8650 1390 50  0001 C CNN
-F 2 "" H 8650 1500 60  0000 C CNN
-F 3 "" H 8650 1500 60  0000 C CNN
-	1    8650 1500
+P 8650 1950
+F 0 "#PWR011" H 8650 1750 50  0001 C CNN
+F 1 "GND" H 8650 1840 50  0001 C CNN
+F 2 "" H 8650 1950 60  0000 C CNN
+F 3 "" H 8650 1950 60  0000 C CNN
+	1    8650 1950
 	1    0    0    -1
 $EndComp
@@
 L GND #PWR013
 U 1 1 55A105FF
-P 9450 3700
-F 0 "#PWR013" H 9450 3500 50  0001 C CNN
-F 1 "GND" H 9450 3590 50  0001 C CNN
-F 2 "" H 9450 3700 60  0000 C CNN
-F 3 "" H 9450 3700 60  0000 C CNN
-	1    9450 3700
-	1    0    0    -1
-$EndComp
-Text Notes 10100 3100 0    60   ~ 0
+P 9300 3750
+F 0 "#PWR013" H 9300 3550 50  0001 C CNN
+F 1 "GND" H 9300 3640 50  0001 C CNN
+F 2 "" H 9300 3750 60  0000 C CNN
+F 3 "" H 9300 3750 60  0000 C CNN
+	1    9300 3750
+	1    0    0    -1
+$EndComp
+Text Notes 10600 3100 0    60   ~ 0
 +24V\n\nA\n\nB \n\nGND
 Entry Wire Line
@@
 	6850 2800 7200 2800
 Wire Wire Line
-	8200 2700 9800 2700
+	8200 2700 10300 2700
 Wire Wire Line
 	8350 2900 8350 3000
@@
 	6750 5800 6750 2750
 Wire Wire Line
-	8350 2900 9800 2900
+	8350 2900 10300 2900
 Wire Wire Line
 	4650 3250 4300 3250
@@
 	7200 1450 7200 1600
 Wire Wire Line
-	9700 2400 9700 2500
-Wire Wire Line
-	9800 3100 9700 3100
+	10300 3100 9700 3100
 Wire Wire Line
 	9700 3100 9700 3650
 Wire Wire Line
-	8650 1100 8650 1200
-Wire Wire Line
-	8650 1200 8550 1200
+	9600 1100 9600 1200
 Wire Wire Line
 	8550 1400 8650 1400
 Wire Wire Line
-	8650 1400 8650 1500
+	8650 1400 8650 1950
 Connection ~ 7200 1500
 Connection ~ 7200 1100
@@
 Wire Wire Line
 	8900 3650 9700 3650
-Connection ~ 9450 3650
 Connection ~ 8550 2700
 Connection ~ 9250 2900
@@
 Wire Wire Line
 	1850 3700 1950 3700
-Wire Wire Line
-	1950 3800 1750 3800
 Wire Bus Line
 	2750 2700 2750 5800
 Wire Bus Line
 	1550 5800 6750 5800
-Wire Wire Line
-	9450 2500 9800 2500
-Wire Wire Line
-	9450 3550 9450 3700
 Wire Wire Line
 	5350 4650 5350 5300
@@
 	0    -1   1    0
 $EndComp
-$Comp
-L +5V #PWR022
-U 1 1 55F77D7B
-P 1750 3800
-F 0 "#PWR022" H 1750 4000 50  0001 C CNN
-F 1 "+5V" H 1750 3910 50  0000 C CNN
-F 2 "" H 1750 3800 60  0000 C CNN
-F 3 "" H 1750 3800 60  0000 C CNN
-	1    1750 3800
-	0    -1   1    0
-$EndComp
 Text Label 2350 2700 0    40   ~ 0
 PC2_INT0
 Wire Wire Line
 	2350 2600 2600 2600
-$Comp
-L +5V #PWR023
-U 1 1 55F78B8C
-P 2550 3800
-F 0 "#PWR023" H 2550 4000 50  0001 C CNN
-F 1 "+5V" H 2550 3910 50  0000 C CNN
-F 2 "" H 2550 3800 60  0000 C CNN
-F 3 "" H 2550 3800 60  0000 C CNN
-	1    2550 3800
-	0    1    1    0
-$EndComp
-Wire Wire Line
-	2550 3800 2350 3800
 $Comp
 L +5V #PWR024
@@
 L Varistor R7
 U 1 1 55F7A87F
-P 9450 3300
-F 0 "R7" H 9295 3210 50  0000 L CNN
-F 1 "Varistor" H 9450 3300 50  0000 C CNN
-F 2 "Resistor:R400" H 9450 3300 60  0001 C CNN
-F 3 "" H 9450 3300 60  0000 C CNN
-	1    9450 3300
-	0    1    1    0
-$EndComp
-Wire Wire Line
-	9450 2500 9450 3050
-Connection ~ 9700 2500
+P 8900 1550
+F 0 "R7" H 8745 1460 50  0000 L CNN
+F 1 "Varistor" H 8900 1550 50  0000 C CNN
+F 2 "Resistor:R400" H 8900 1550 60  0001 C CNN
+F 3 "" H 8900 1550 60  0000 C CNN
+	1    8900 1550
+	0    1    1    0
+$EndComp
 Wire Wire Line
 	7200 2900 7100 2900
@@
 F 0 "D2" H 8975 3050 50  0000 C CNN
 F 1 "SEMTECH_SR05" H 8900 3550 50  0000 C CNN
-F 2 "Housings_SOT:SOT143R_Diode_Reverse" H 8900 3300 60  0001 C CNN
+F 2 "Diode_SMD:SOT143" H 8900 3300 60  0001 C CNN
 F 3 "" H 8900 3300 60  0000 C CNN
 	1    8900 3300
@@
 Text Label 9000 2900 0    40   ~ 0
 B
+$Comp
+L FUSE F1
+U 1 1 56645547
+P 9200 1200
+F 0 "F1" H 9200 1300 50  0000 C CNN
+F 1 "FUSE" H 9200 1100 50  0000 C CNN
+F 2 "Resistor:R_1812" H 9200 1200 60  0001 C CNN
+F 3 "" H 9200 1200 60  0000 C CNN
+	1    9200 1200
+	1    0    0    -1
+$EndComp
+$Comp
+L +24V #PWR?
+U 1 1 5AB96AC4
+P 2550 3800
+F 0 "#PWR?" H 2550 4000 50  0001 C CNN
+F 1 "+24V" H 2550 3910 50  0000 C CNN
+F 2 "" H 2550 3800 60  0000 C CNN
+F 3 "" H 2550 3800 60  0000 C CNN
+	1    2550 3800
+	0    1    1    0
+$EndComp
+$Comp
+L +24V #PWR?
+U 1 1 5AB96BDD
+P 1750 3800
+F 0 "#PWR?" H 1750 4000 50  0001 C CNN
+F 1 "+24V" H 1750 3910 50  0000 C CNN
+F 2 "" H 1750 3800 60  0000 C CNN
+F 3 "" H 1750 3800 60  0000 C CNN
+	1    1750 3800
+	0    -1   1    0
+$EndComp
+Wire Wire Line
+	1750 3800 1950 3800
+Wire Wire Line
+	2350 3800 2550 3800
+Wire Wire Line
+	9000 1200 8550 1200
+Wire Wire Line
+	9600 1200 9400 1200
+Wire Wire Line
+	8900 1300 8900 1200
+Connection ~ 8900 1200
+Wire Wire Line
+	8900 1800 8900 1900
+Wire Wire Line
+	8900 1900 8650 1900
+Connection ~ 8650 1900
+Wire Wire Line
+	10300 2500 10100 2500
+Wire Wire Line
+	10100 2500 10100 2400
+Wire Wire Line
+	9300 3750 9300 3650
+Connection ~ 9300 3650
 $EndSCHEMATC

Commit message: Finalized revB of bus-module_attiny1634
Parts:
- removed F1: FUSE, Resistor:R_1812, symbol FUSE
- removed U3: ATtiny1634-SOIC, Housings_SOIC:SO20L, symbol ATtiny1634-SOIC
- removed U5: AM1S-2403, DCDC_Converter:AM1S-XXXX_SIL4, symbol AM1S-2403
- added F1: FUSE, symbol standard:FUSE
- added U3: ATTINY1634-SOIC, SO20L, symbol ics_controller_atmel:ATTINY1634-SOIC
- added U5: AM1S-2405, AM1S-XXXX_SIL4, symbol ics_regulator:AM1S-2405
- C1, C2, C3, C4, C5, C7: symbol C -> standard:C
- C6: symbol CP -> standard:CP
- D1: symbol D -> standard:D
- D2: symbol SEMTECH_SR05 -> diodes:SEMTECH_SR05
- H1: symbol HOLE -> standard:HOLE
- J1, J2: symbol CONN_5X2 -> connectors:CONN_5X2
- J3: symbol CONN-ISP-6 -> connectors:CONN-ISP-6
- J4, J5, J6, J7: symbol CONN_1 -> connectors:CONN_1
- LOGO1: symbol OPEN_HARDWARE_1 -> logo:OPEN_HARDWARE_1
- R1, R2, R3, R4, R5, R6: symbol R -> standard:R
- R7: symbol Varistor -> standard:Varistor
- U1: symbol CRYSTAL -> standard:CRYSTAL
- U2: symbol 25LCXXX -> ics_peripheral:25LCXXX
- U4: symbol MAX487 -> ics_misc:MAX487
Connections:
- net +24V: now also F1.2
- net /CSEEP: now also U3.17 (PC0/OC0A)
- net /RESET: now also U3.14 (PC3/RESETn)
- net GND: now also U3.10 (GND), U5.1 (VIN-), U5.3 (VOUT-)
- net PA0_AREF: now also U3.9 (PA0/AREF)
- net PA1: now also U3.8 (PA1/AIN0)
- net PA2: now also U3.7 (PA2/AIN1)
- net PA3: now also U3.6 (PA3/T1)
- net PA4: now also U3.5 (PA4/T0)
- net PA5: now also U3.4 (PA5/OC0B)
- net PB1_MISO: now also U3.20 (PB1/RXD1)
- net PB2_MOSI: now also U3.19 (PB2/TXD1)
- net PB3: now also U3.18 (PB3/OC1A)
- net PC1_SCK: now also U3.16 (PC1/SCL)
- net PC2_INT0: now also U3.15 (PC2)
- net RXD: now also U3.2 (PA7/RXD0)
- net TXD: now also U3.1 (PB0/TXD0)
- net TXDEN: now also U3.3 (PA6/OC1B)
- net at R7.1: now also F1.1, U5.2 (VIN+)
- net at C3.1, U1.2: now also U3.13 (PC4/XTAL2)
- net at C2.1, U1.1: now also U3.12 (PC5/XTAL1)
- net +5V renamed VCC
- net VCC: now also U3.11 (VCC), U5.4 (VOUT+)
