File: hw/motor_switch_3pole_5x/bus_atmega328_basic.sch (KiCad schematic (older format))
At the start: 26 parts, among them J12 CONN-ISP-6, J13 WAGO 243-723, J14 WAGO 243-724, J15 WAGO 243-721, J16 WAGO 243-722, U3 25LC256, U4 ATMEGA328-TQFP32, U5 7,3728MHz, U6 MAX487ECSA, U7 AM1S-2405

Commit message: added LEDs and testpoints to PCB
Parts:
- added J29: tp_cseep, Connector_Miscelleaneus:Testpoint_1mm, symbol connectors:CONN_1
- added J30: tp_vcc, Connector_Miscelleaneus:Testpoint_1mm, symbol connectors:CONN_1
- added J31: tp_gnd, Connector_Miscelleaneus:Testpoint_1mm, symbol connectors:CONN_1
- added J46: tp_miso, Connector_Miscelleaneus:Testpoint_1mm, symbol connectors:CONN_1
- added J47: tp_txden, Connector_Miscelleaneus:Testpoint_1mm, symbol connectors:CONN_1
- added J48: tp_txd, Connector_Miscelleaneus:Testpoint_1mm, symbol connectors:CONN_1
- added J49: tp_rxd, Connector_Miscelleaneus:Testpoint_1mm, symbol connectors:CONN_1
- C3, C4, C5, C6, C7, C8, C9: symbol C -> standard:C
- D22: symbol SEMTECH_SR05 -> diodes:SEMTECH_SR05
- F2: symbol FUSE -> standard:FUSE
- J12: symbol CONN-ISP-6 -> connectors:CONN-ISP-6
- J13, J14, J15, J16: symbol CONN_1 -> connectors:CONN_1
- LOGO4: symbol OPEN_HARDWARE_1 -> logo:OPEN_HARDWARE_1
- R31, R32, R33, R34, R35, R36: symbol R -> standard:R
- U3: symbol 25LCXXX -> ics_peripheral:25LCXXX
- U4: symbol ATMEGA88-TQFP32 -> ics_controller_atmel:ATMEGA88-TQFP32
- U5: symbol CRYSTAL -> standard:CRYSTAL
- U6: symbol MAX487 -> ics_misc:MAX487
- U7: symbol AM1S-2403 -> ics_regulator:AM1S-2403
Connections:
- net /CSEEP: now also J29.1
- net GND: now also J31.1
- net MISO: now also J46.1
- net RXD0: now also J49.1
- net TXD0: now also J48.1
- net TXD0EN: now also J47.1
- net VCC: now also J30.1
