File: hw/motor_switch_3pole_5x/bus_atmega328_basic.sch (KiCad schematic (older format))
At the start: 33 parts, among them J12 CONN-ISP-6, J13 WAGO 243-723, J14 WAGO 243-724, J15 WAGO 243-721, J16 WAGO 243-722, J29 tp_cseep, J30 tp_vcc, J31 tp_gnd, J46 tp_miso, J47 tp_txden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

Commit message: Update to revision B. Fixed footprint of U4
Parts:
- U4: footprint Housings_QFP:TQFP-44_10x10mm_Pitch0.8mm -> Housings_QFP:TQFP-32_7x7mm_Pitch0.8mm
Changed lines of the file:
@@
 Sheet 4 4
 Title "motor switch 3pole (bus_atmega328_basic)"
-Date "2018-09-18"
-Rev "A"
+Date "2018-12-27"
+Rev "B"
 Comp "KoeWiBa"
 Comment1 ""
@@
 F 0 "U4" H 5350 3550 50  0000 C CNN
 F 1 "ATMEGA328-TQFP32" H 5350 2750 50  0000 C CNN
-F 2 "Housings_QFP:TQFP-44_10x10mm_Pitch0.8mm" H 5350 3550 25  0001 C CNN
+F 2 "Housings_QFP:TQFP-32_7x7mm_Pitch0.8mm" H 5350 3550 25  0001 C CNN
 F 3 "DOCUMENTATION" H 5350 3550 25  0001 C CNN
 	1    5350 3550
