File: hw/motor_switch_3pole_5x/inputs.sch (KiCad schematic (older format))
At the start: 27 parts, among them J10 WAGO 233-504, J11 WAGO 233-504, J7 WAGO 233-504, J8 WAGO 233-504, J9 WAGO 233-504

Commit message: added LEDs and testpoints to PCB
Parts:
- added J32: tp_output_button_0_up, Connector_Miscelleaneus:Testpoint_1mm, symbol connectors:CONN_1
- added J33: tp_output_button_0_down, Connector_Miscelleaneus:Testpoint_1mm, symbol connectors:CONN_1
- added J34: tp_output_button_1_up, Connector_Miscelleaneus:Testpoint_1mm, symbol connectors:CONN_1
- added J35: tp_output_button_1_down, Connector_Miscelleaneus:Testpoint_1mm, symbol connectors:CONN_1
- added J36: tp_output_button_2_up, Connector_Miscelleaneus:Testpoint_1mm, symbol connectors:CONN_1
- added J37: tp_output_button_2_down, Connector_Miscelleaneus:Testpoint_1mm, symbol connectors:CONN_1
- added J38: tp_output_button_3_up, Connector_Miscelleaneus:Testpoint_1mm, symbol connectors:CONN_1
- added J39: tp_output_button_3_down, Connector_Miscelleaneus:Testpoint_1mm, symbol connectors:CONN_1
- added J40: tp_output_button_4_up, Connector_Miscelleaneus:Testpoint_1mm, symbol connectors:CONN_1
- added J41: tp_output_button_4_down, Connector_Miscelleaneus:Testpoint_1mm, symbol connectors:CONN_1
- D11, D12, D13, D14, D15, D16, D17, D18, D19, D20: symbol BAT54S -> diodes:BAT54S
- D21: symbol ZD -> standard:ZD
- J10, J11, J7, J8, J9: symbol CONN_4X1 -> connectors:CONN_4X1
- LOGO3: symbol OPEN_HARDWARE_1 -> logo:OPEN_HARDWARE_1
- R21, R22, R23, R24, R25, R26, R27, R28, R29, R30: symbol R -> standard:R
Connections:
- net button_0_down: now also J33.1
- net button_0_up: now also J32.1
- net button_1_down: now also J35.1
- net button_1_up: now also J34.1
- net button_2_down: now also J37.1
- net button_2_up: now also J36.1
- net button_3_down: now also J39.1
- net button_3_up: now also J38.1
- net button_4_down: now also J41.1
- net button_4_up: now also J40.1
