File: hw/motor_switch_3pole_5x/motor_relays.sch (KiCad schematic (older format))
At the start: 59 parts, among them J1 CONN_2X1, J17 CONN_1, J18 CONN_1, J2 WAGO 2081-1122, J3 WAGO 2081-1122, J4 WAGO 2081-1122, J5 WAGO 2081-1122, J6 WAGO 2081-1122, Q1 BSS138, Q10 BSS138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

Commit message: added LEDs and testpoints to PCB
Parts:
- added D23, D25, D27, D29, D31: yellow, 2,1V/2mA, LED:LED_RM2.54mm_D3mm, symbol standard:LED
- added D24, D26, D28, D30, D32: green, 2,2V/2mA, LED:LED_RM2.54mm_D3mm, symbol standard:LED
- added J19: tp_output_motor_0_up, Connector_Miscelleaneus:Testpoint_1mm, symbol connectors:CONN_1
- added J20: tp_output_motor_on, Connector_Miscelleaneus:Testpoint_1mm, symbol connectors:CONN_1
- added J21: tp_output_motor_1_up, Connector_Miscelleaneus:Testpoint_1mm, symbol connectors:CONN_1
- added J22: tp_output_motor_1_on, Connector_Miscelleaneus:Testpoint_1mm, symbol connectors:CONN_1
- added J23: tp_output_motor_2_up, Connector_Miscelleaneus:Testpoint_1mm, symbol connectors:CONN_1
- added J24: tp_output_motor_2_on, Connector_Miscelleaneus:Testpoint_1mm, symbol connectors:CONN_1
- added J25: tp_output_motor_3_up, Connector_Miscelleaneus:Testpoint_1mm, symbol connectors:CONN_1
- added J26: tp_output_motor_3_on, Connector_Miscelleaneus:Testpoint_1mm, symbol connectors:CONN_1
- added J27: tp_output_motor_4_up, Connector_Miscelleaneus:Testpoint_1mm, symbol connectors:CONN_1
- added J28: tp_output_motor_4_on, Connector_Miscelleaneus:Testpoint_1mm, symbol connectors:CONN_1
- added R37, R38, R39, R40, R41, R42, R43, R44, R45, R46: 1k5, Resistor:R_0805, symbol standard:R
- D1, D10, D2, D3, D4, D5, D6, D7, D8, D9: symbol D -> standard:D
- J1, J2, J3, J4, J5, J6: symbol CONN_2X1 -> connectors:CONN_2X1
- J17, J18: symbol CONN_1 -> connectors:CONN_1
- LOGO2: symbol OPEN_HARDWARE_1 -> logo:OPEN_HARDWARE_1
- Q1, Q10, Q2, Q3, Q4, Q5, Q6, Q7, Q8, Q9: symbol BSS138 -> transistors:BSS138
- R1, R10, R11, R12, R13, R14, R15, R16, R17, R18, R19, R2, R20, R3, R4, R5, R6, R7, R8, R9: symbol R -> standard:R
- REL1, REL10, REL2, REL3, REL4, REL5, REL6, REL7, REL8, REL9: symbol FINDER_34.51.7.024 -> relays:FINDER_34.51.7.024
Connections:
- net at D1.1 (A), Q1.3 (D), REL1.1 (+): now also D23.2 (C), J19.1
- net at D2.1 (A), Q2.3 (D), REL2.1 (+): now also D24.2 (C), J20.1
- net at D3.1 (A), Q3.3 (D), REL3.1 (+): now also D25.2 (C), J21.1
- net at D4.1 (A), Q4.3 (D), REL4.1 (+): now also D26.2 (C), J22.1
- net at D7.1 (A), Q7.3 (D), REL7.1 (+): now also D29.2 (C), J25.1
- net at D8.1 (A), Q8.3 (D), REL8.1 (+): now also D30.2 (C), J26.1
- net at D9.1 (A), Q9.3 (D), REL9.1 (+): now also D31.2 (C), J27.1
- net at D10.1 (A), Q10.3 (D), REL10.1 (+): now also D32.2 (C), J28.1
- net at D5.1 (A), Q5.3 (D), REL5.1 (+): now also D27.2 (C), J23.1
- net at D6.1 (A), Q6.3 (D), REL6.1 (+): now also D28.2 (C), J24.1
- new net: D23.1 (A), R37.1
- new net: D24.1 (A), R38.1
- new net: D25.1 (A), R39.1
- new net: D26.1 (A), R40.1
- new net: D27.1 (A), R41.1
- new net: D28.1 (A), R42.1
- new net: D29.1 (A), R43.1
- new net: D30.1 (A), R44.1
- new net: D31.1 (A), R45.1
- new net: D32.1 (A), R46.1
- new net +5V: R37.2, R38.2, R39.2, R40.2, R41.2, R42.2, R43.2, R44.2, R45.2, R46.2
Other:
- moved on the sheet: D1, D10, D2, D3, D4, D5, D6, D7, D8, D9, J2, J3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
