File: hw/motor_switch_3pole_5x/motor_switch_3pole_5x.sch (KiCad schematic (older format))
At the start: 5 parts, among them U1 74HC595, U2 74HC595

Commit message: added LEDs and testpoints to PCB
Parts:
- added J42: tp_output_latch, Connector_Miscelleaneus:Testpoint_1mm, symbol connectors:CONN_1
- added J43: tp_output_data, Connector_Miscelleaneus:Testpoint_1mm, symbol connectors:CONN_1
- added J44: tp_output_clock, Connector_Miscelleaneus:Testpoint_1mm, symbol connectors:CONN_1
- added J45: tp_output_reset, Connector_Miscelleaneus:Testpoint_1mm, symbol connectors:CONN_1
- C1, C2: symbol C -> standard:C
- LOGO1: symbol OPEN_HARDWARE_1 -> logo:OPEN_HARDWARE_1
- U1, U2: symbol 74HC595 -> ics_74xx:74HC595
Connections:
- net output_clock: now also J44.1
- net output_data: now also J43.1
- net output_latch: now also J42.1
- net output_reset: now also J45.1
Changed lines of the file:
@@
-EESchema Schematic File Version 2
-LIBS:diodes
-LIBS:ics_controller_atmel
-LIBS:ics_misc
-LIBS:ics_peripheral
-LIBS:logo
-LIBS:analog_devices
-LIBS:connectors
-LIBS:display
-LIBS:encoder
-LIBS:ftdi
-LIBS:ics_40xx
-LIBS:ics_74xx
-LIBS:ics_opamp
-LIBS:ics_opto
-LIBS:ics_regulator
-LIBS:ics_signal
-LIBS:modules
-LIBS:power
-LIBS:relays
-LIBS:sensors
-LIBS:standard
-LIBS:transformer
-LIBS:transistors
+EESchema Schematic File Version 4
 LIBS:motor_switch_3pole_5x-cache
-EELAYER 25 0
+EELAYER 26 0
 EELAYER END
 $Descr A4 11693 8268
@@
 Sheet 1 4
 Title "motor switch 3pole 5x"
-Date "2018-06-07"
+Date "2018-09-17"
 Rev "1"
 Comp "koewiba"
@@
 $EndDescr
 $Comp
-L +5V #PWR01
+L power:+5V #PWR01
 U 1 1 572DAEDB
 P 4300 3050
@@
 $EndComp
 $Comp
-L +24V #PWR02
+L power:+24V #PWR02
 U 1 1 572DAF09
 P 2600 3050
@@
 $EndComp
 $Comp
-L OPEN_HARDWARE_1 LOGO1
+L logo:OPEN_HARDWARE_1 LOGO1
 U 1 1 572E288C
 P 1025 7400
@@
 $EndSheet
 $Comp
-L GND #PWR03
+L power:GND #PWR03
 U 1 1 578B8717
 P 4300 4600
@@
 $EndSheet
 $Comp
-L 74HC595 U2
+L ics_74xx:74HC595 U2
 U 1 1 5B0E7E5B
 P 8300 3800
@@
 $EndComp
 $Comp
-L 74HC595 U1
+L ics_74xx:74HC595 U1
 U 1 1 5B0EF04A
 P 6200 3800
@@
 $EndComp
 $Comp
-L C C2
+L standard:C C2
 U 1 1 5B0F03CD
 P 8100 2950
@@
 $EndComp
 $Comp
-L C C1
+L standard:C C1
 U 1 1 5B0F0568
 P 6000 2950
@@
 $EndComp
 $Comp
-L +5V #PWR04
+L power:+5V #PWR04
 U 1 1 5B0F0960
 P 8300 2750
@@
 $EndComp
 $Comp
-L +5V #PWR05
+L power:+5V #PWR05
 U 1 1 5B0F0D67
 P 6200 2750
@@
 $EndComp
 $Comp
-L GND #PWR06
+L power:GND #PWR06
 U 1 1 5B0F16A2
 P 6000 3150
@@
 $EndComp
 $Comp
-L GND #PWR07
+L power:GND #PWR07
 U 1 1 5B0F17D2
 P 8100 3150
@@
 NoConn ~ 8900 4250
 $Comp
-L GND #PWR08
+L power:GND #PWR08
 U 1 1 5B0F354D
 P 8300 4650
@@
 $EndComp
 $Comp
-L GND #PWR09
+L power:GND #PWR09
 U 1 1 5B0F3C09
 P 6200 4650
@@
 	6000 2850 6200 2850
 Wire Wire Line
-	6200 2750 6200 3050
+	6200 2750 6200 2850
 Connection ~ 6200 2850
 Wire Wire Line
-	8300 2750 8300 3050
+	8300 2750 8300 2850
 Wire Wire Line
 	8100 2850 8300 2850
@@
 	6000 3050 6000 3150
 Wire Wire Line
-	6200 4550 6200 4650
-Wire Wire Line
-	8300 4550 8300 4650
+	6200 4550 6200 4600
+Wire Wire Line
+	8300 4550 8300 4600
 Wire Wire Line
 	6800 3350 7150 3350
@@
 Wire Wire Line
 	6800 4050 7150 4050
-Wire Bus Line
-	7250 3450 7250 4900
 Wire Wire Line
 	10100 3350 9650 3350
@@
 Wire Wire Line
 	10100 4450 9650 4450
-Wire Bus Line
-	9550 4900 9550 3450
 Wire Wire Line
 	6800 4250 7350 4250
@@
 	5450 4850 5450 3850
 Wire Wire Line
-	4950 3850 5600 3850
-Wire Wire Line
-	4950 3650 5600 3650
+	4950 3850 5450 3850
+Wire Wire Line
+	4950 3650 5400 3650
 Wire Wire Line
 	5400 3650 5400 4800
@@
 	5350 4750 5350 3550
 Wire Wire Line
-	4950 3550 5600 3550
+	4950 3550 5350 3550
 Text Label 1600 3150 0    40   ~ 0
 /button_0_up
@@
 Wire Wire Line
 	2600 3800 3100 3800
-Wire Bus Line
-	4650 4750 4650 3400
-Wire Bus Line
-	2500 4750 2500 3600
-Wire Bus Line
-	2200 3250 2200 4750
 Text Label 4050 3950 0    40   ~ 0
 output_data
@@
 Wire Wire Line
 	4000 4350 4450 4350
-Wire Bus Line
-	2400 3350 2400 4850
-Wire Bus Line
-	4550 4850 4550 4050
 Entry Wire Line
 	4850 3450 4950 3350
@@
 Connection ~ 5450 3850
 Wire Bus Line
-	4850 4850 4850 3450
-Wire Bus Line
 	2200 4750 4650 4750
-Wire Bus Line
-	2400 4850 4850 4850
 Text Label 2950 4850 0    40   ~ 0
 output
@@
 Wire Wire Line
 	8900 4050 9250 4050
+Wire Wire Line
+	6200 2850 6200 3050
+Wire Wire Line
+	8300 2850 8300 3050
+Wire Wire Line
+	8300 4600 8300 4650
+Wire Wire Line
+	6200 4600 6200 4650
+Wire Wire Line
+	5350 3550 5600 3550
+Wire Wire Line
+	5400 3650 5600 3650
+Wire Wire Line
+	5450 3850 5600 3850
+Entry Wire Line
+	2400 4950 2500 5050
+Entry Wire Line
+	2400 5050 2500 5150
+Entry Wire Line
+	2400 5150 2500 5250
+Entry Wire Line
+	2400 5250 2500 5350
+Text Label 2550 5050 0    40   ~ 0
+output_latch
+Text Label 2550 5150 0    40   ~ 0
+output_data
+Text Label 2550 5250 0    40   ~ 0
+output_clock
+Text Label 2550 5350 0    40   ~ 0
+output_reset
+Wire Wire Line
+	2950 5050 2500 5050
+Wire Wire Line
+	2500 5150 2950 5150
+Wire Wire Line
+	2500 5250 2950 5250
+Wire Wire Line
+	2500 5350 2950 5350
+Wire Bus Line
+	2400 4850 4850 4850
+Connection ~ 2400 4850
+Wire Bus Line
+	2400 3350 2400 4850
+$Comp
+L connectors:CONN_1 J42
+U 1 1 5BA1D0CF
+P 3050 5050
+F 0 "J42" H 3091 5086 50  0000 L CNN
+F 1 "tp_output_latch" H 3250 5050 25  0000 L CNN
+F 2 "Connector_Miscelleaneus:Testpoint_1mm" H 3050 5050 60  0001 C CNN
+F 3 "" H 3050 5050 60  0000 C CNN
+	1    3050 5050
+	1    0    0    -1
+$EndComp
+$Comp
+L connectors:CONN_1 J43
+U 1 1 5BA1D111
+P 3050 5150
+F 0 "J43" H 3091 5186 50  0000 L CNN
+F 1 "tp_output_data" H 3250 5150 25  0000 L CNN
+F 2 "Connector_Miscelleaneus:Testpoint_1mm" H 3050 5150 60  0001 C CNN
+F 3 "" H 3050 5150 60  0000 C CNN
+	1    3050 5150
+	1    0    0    -1
+$EndComp
+$Comp
+L connectors:CONN_1 J44
+U 1 1 5BA1D14E
+P 3050 5250
+F 0 "J44" H 3091 5286 50  0000 L CNN
+F 1 "tp_output_clock" H 3250 5250 25  0000 L CNN
+F 2 "Connector_Miscelleaneus:Testpoint_1mm" H 3050 5250 60  0001 C CNN
+F 3 "" H 3050 5250 60  0000 C CNN
+	1    3050 5250
+	1    0    0    -1
+$EndComp
+$Comp
+L connectors:CONN_1 J45
+U 1 1 5BA1D18E
+P 3050 5350
+F 0 "J45" H 3091 5386 50  0000 L CNN
+F 1 "tp_output_reset" H 3250 5350 25  0000 L CNN
+F 2 "Connector_Miscelleaneus:Testpoint_1mm" H 3050 5350 60  0001 C CNN
+F 3 "" H 3050 5350 60  0000 C CNN
+	1    3050 5350
+	1    0    0    -1
+$EndComp
 Wire Bus Line
 	9350 4050 9350 4900
+Wire Bus Line
+	4550 4050 4550 4850
+Wire Bus Line
+	4850 3450 4850 4850
+Wire Bus Line
+	2500 3600 2500 4750
+Wire Bus Line
+	2400 4850 2400 5250
+Wire Bus Line
+	4650 3400 4650 4750
+Wire Bus Line
+	9550 3450 9550 4900
+Wire Bus Line
+	2200 3250 2200 4750
+Wire Bus Line
+	7250 3450 7250 4900
 $EndSCHEMATC
