File: hw/bus-module_atmega324/bus-module_atmega324.sch (KiCad schematic (older format))
At the start: 35 parts, among them J1 CONN_10X2, J2 CONN_10X2, J3 CONN-ISP-6, J5 CONN_1, J6 CONN_1, J7 CONN_1, J8 CONN_1, U1 ATMEGA324-TQFP44, U2 7,3728MHz, U3 25LCXXX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

Commit message: added bus-module_atmega324 rev B
Parts:
- added F1: FUSE, Resistor:R_1812, symbol bus-module_atmega324-rescue:FUSE
- C1, C10, C11, C2, C3, C4, C5, C6, C7, C8: symbol C -> standard:C
- C9: symbol CP -> standard:CP
- D1: symbol D -> standard:D
- D2: footprint Housings_SOT:SOT143R_Diode_Reverse -> Diode_SMD:SOT143; symbol SEMTECH_SR05 -> diodes:SEMTECH_SR05
- H1: symbol HOLE -> standard:HOLE
- J1, J2: symbol CONN_10X2-RESCUE-bus-module_atmega324 -> bus-module_atmega324-rescue:CONN_10X2-RESCUE-bus-module_atmega324
- J3: symbol CONN-ISP-6 -> connectors:CONN-ISP-6
- J5, J6, J7, J8: symbol CONN_1 -> connectors:CONN_1
- L1: symbol L -> standard:L
- LOGO1: symbol OPEN_HARDWARE_1 -> logo:OPEN_HARDWARE_1
- R1, R2, R3, R4, R5, R6: symbol R -> standard:R
- U1: symbol ATMEGA324-TQFP44 -> ics_controller_atmel:ATMEGA324-TQFP44
- U2: symbol CRYSTAL -> standard:CRYSTAL
- U3: symbol 25LCXXX -> ics_peripheral:25LCXXX
- U4, U5: symbol MAX487 -> ics_misc:MAX487
- U6: symbol AM1S-2403 -> ics_regulator:AM1S-2403
Connections:
- net +24V: now also J1.3, J1.4, F1.2; no longer U6.2 (VIN+)
- net +3.3V: no longer J1.3, J1.4
- new net: F1.1, U6.2 (VIN+)

Commit message: changed 3,3V net to VCC net changed silkscreen description of pins removed need of rescue lib
Parts:
- F1: symbol bus-module_atmega324-rescue:FUSE -> standard:FUSE
- J1, J2: symbol bus-module_atmega324-rescue:CONN_10X2-RESCUE-bus-module_atmega324 -> connectors:CONN_10X2
Connections:
- net labels added: VCC
- net labels removed: +3.3V
Changed lines of the file:
@@
 Sheet 1 1
 Title "bus-module_atmega324"
-Date "2018-09-23"
+Date "2018-09-24"
 Rev "B"
 Comp "KoeWiBa"
@@
 $EndComp
 $Comp
-L power:+3.3V #PWR05
-U 1 1 559D7883
-P 7600 2100
-F 0 "#PWR05" H 7600 2300 50  0001 C CNN
-F 1 "+3.3V" H 7600 2210 50  0000 C CNN
-F 2 "" H 7600 2100 60  0000 C CNN
-F 3 "" H 7600 2100 60  0000 C CNN
-	1    7600 2100
-	1    0    0    -1
-$EndComp
-$Comp
-L power:+3.3V #PWR06
-U 1 1 559D7915
-P 4850 1400
-F 0 "#PWR06" H 4850 1600 50  0001 C CNN
-F 1 "+3.3V" H 4850 1510 50  0000 C CNN
-F 2 "" H 4850 1400 60  0000 C CNN
-F 3 "" H 4850 1400 60  0000 C CNN
-	1    4850 1400
-	1    0    0    -1
-$EndComp
-$Comp
 L standard:R R4
 U 1 1 559D7BAA
@@
 F 3 "" H 8000 3900 60  0000 C CNN
 	1    8000 3900
-	1    0    0    -1
-$EndComp
-$Comp
-L power:+3.3V #PWR010
-U 1 1 55A00E8D
-P 7600 3700
-F 0 "#PWR010" H 7600 3900 50  0001 C CNN
-F 1 "+3.3V" H 7600 3810 50  0000 C CNN
-F 2 "" H 7600 3700 60  0000 C CNN
-F 3 "" H 7600 3700 60  0000 C CNN
-	1    7600 3700
 	1    0    0    -1
 $EndComp
@@
 PB6_MISO
 $Comp
-L power:+3.3V #PWR013
-U 1 1 55A085DC
-P 8000 5400
-F 0 "#PWR013" H 8000 5600 50  0001 C CNN
-F 1 "+3.3V" H 8000 5510 50  0000 C CNN
-F 2 "" H 8000 5400 60  0000 C CNN
-F 3 "" H 8000 5400 60  0000 C CNN
-	1    8000 5400
-	1    0    0    -1
-$EndComp
-$Comp
 L power:GND #PWR014
 U 1 1 55A08693
@@
 U 1 1 55A0D0CD
 P 6350 2250
-F 0 "C7" H 6400 2300 50  0000 L CNN
+F 0 "C7" H 6400 2325 50  0000 L CNN
 F 1 "100nF" H 6500 2200 50  0000 C CNN
 F 2 "Housings_SOIC:SM0805" H 6350 2250 60  0001 C CNN
@@
 U 1 1 55A0D462
 P 6550 2250
-F 0 "C8" H 6600 2300 50  0000 L CNN
-F 1 "4,7nF" H 6650 2400 50  0000 C CNN
+F 0 "C8" H 6600 2325 50  0000 L CNN
+F 1 "4,7nF" H 6700 2400 50  0000 C CNN
 F 2 "Housings_SOIC:SM0805" H 6550 2250 60  0001 C CNN
 F 3 "" H 6550 2250 60  0000 C CNN
@@
 	8650 1400 8650 1500
 Connection ~ 7200 1500
-$Comp
-L power:+3.3V #PWR021
-U 1 1 55A113A0
-P 7200 1000
-F 0 "#PWR021" H 7200 1200 50  0001 C CNN
-F 1 "+3.3V" H 7200 1110 50  0000 C CNN
-F 2 "" H 7200 1000 60  0000 C CNN
-F 3 "" H 7200 1000 60  0000 C CNN
-	1    7200 1000
-	1    0    0    -1
-$EndComp
 Connection ~ 7200 1100
 Text Notes 10100 3100 0    60   ~ 0
@@
 Wire Wire Line
 	6200 4450 6650 4450
-$Comp
-L power:+3.3V #PWR022
-U 1 1 55A147BE
-P 1850 2600
-F 0 "#PWR022" H 1850 2800 50  0001 C CNN
-F 1 "+3.3V" V 1850 2800 50  0000 C CNN
-F 2 "" H 1850 2600 60  0000 C CNN
-F 3 "" H 1850 2600 60  0000 C CNN
-	1    1850 2600
-	0    -1   -1   0
-$EndComp
 $Comp
 L power:GND #PWR023
@@
 Text Label 4300 3850 0    40   ~ 0
 PB1
-$Comp
-L power:+3.3V #PWR025
-U 1 1 55A16808
-P 5400 6050
-F 0 "#PWR025" H 5400 6250 50  0001 C CNN
-F 1 "+3.3V" H 5400 6200 50  0000 C CNN
-F 2 "" H 5400 6050 60  0000 C CNN
-F 3 "" H 5400 6050 60  0000 C CNN
-	1    5400 6050
-	1    0    0    -1
-$EndComp
 Connection ~ 5400 6100
 Text Label 6250 2050 0    40   ~ 0
@@
 P 6750 1750
 F 0 "D1" H 6760 1830 50  0000 C CNN
-F 1 "1N4148WS (SOD323)" H 6750 1675 50  0000 C CNN
+F 1 "1N4148WS (SOD323)" H 6750 1650 50  0000 C CNN
 F 2 "Diode:SOD323" H 6750 1750 60  0001 C CNN
 F 3 "" H 6750 1750 60  0000 C CNN
@@
 B
 $Comp
-L bus-module_atmega324-rescue:CONN_10X2-RESCUE-bus-module_atmega324 J2
+L connectors:CONN_10X2 J2
 U 1 1 56050AF8
 P 2150 2950
@@
 $EndComp
 $Comp
-L bus-module_atmega324-rescue:CONN_10X2-RESCUE-bus-module_atmega324 J1
+L connectors:CONN_10X2 J1
 U 1 1 56050B83
 P 2150 4150
@@
 $EndComp
 $Comp
-L bus-module_atmega324-rescue:FUSE F1
+L standard:FUSE F1
 U 1 1 566474AD
 P 8900 1200
@@
 Wire Wire Line
 	6550 1450 6750 1450
+$Comp
+L power:VCC #PWR0101
+U 1 1 5BAA23B8
+P 1850 2600
+F 0 "#PWR0101" H 1850 2775 50  0001 C CNN
+F 1 "VCC" V 1854 2698 50  0000 L CNN
+F 2 "" H 1850 2600 60  0001 C CNN
+F 3 "" H 1850 2600 60  0001 C CNN
+	1    1850 2600
+	0    -1   -1   0
+$EndComp
+$Comp
+L power:VCC #PWR0102
+U 1 1 5BAA25F3
+P 4850 1400
+F 0 "#PWR0102" H 4850 1575 50  0001 C CNN
+F 1 "VCC" H 4853 1544 50  0000 C CNN
+F 2 "" H 4850 1400 60  0001 C CNN
+F 3 "" H 4850 1400 60  0001 C CNN
+	1    4850 1400
+	1    0    0    -1
+$EndComp
+$Comp
+L power:VCC #PWR0103
+U 1 1 5BAA26A2
+P 7200 1000
+F 0 "#PWR0103" H 7200 1175 50  0001 C CNN
+F 1 "VCC" H 7203 1144 50  0000 C CNN
+F 2 "" H 7200 1000 60  0001 C CNN
+F 3 "" H 7200 1000 60  0001 C CNN
+	1    7200 1000
+	1    0    0    -1
+$EndComp
+$Comp
+L power:VCC #PWR0104
+U 1 1 5BAA2823
+P 7600 2100
+F 0 "#PWR0104" H 7600 2275 50  0001 C CNN
+F 1 "VCC" H 7603 2244 50  0000 C CNN
+F 2 "" H 7600 2100 60  0001 C CNN
+F 3 "" H 7600 2100 60  0001 C CNN
+	1    7600 2100
+	1    0    0    -1
+$EndComp
+$Comp
+L power:VCC #PWR0105
+U 1 1 5BAA29A4
+P 7600 3700
+F 0 "#PWR0105" H 7600 3875 50  0001 C CNN
+F 1 "VCC" H 7500 3750 50  0000 C CNN
+F 2 "" H 7600 3700 60  0001 C CNN
+F 3 "" H 7600 3700 60  0001 C CNN
+	1    7600 3700
+	1    0    0    -1
+$EndComp
+$Comp
+L power:VCC #PWR0106
+U 1 1 5BAA2B52
+P 8000 5400
+F 0 "#PWR0106" H 8000 5575 50  0001 C CNN
+F 1 "VCC" H 8003 5544 50  0000 C CNN
+F 2 "" H 8000 5400 60  0001 C CNN
+F 3 "" H 8000 5400 60  0001 C CNN
+	1    8000 5400
+	1    0    0    -1
+$EndComp
+$Comp
+L power:VCC #PWR0107
+U 1 1 5BAA2CD3
+P 5400 6050
+F 0 "#PWR0107" H 5400 6225 50  0001 C CNN
+F 1 "VCC" H 5403 6194 50  0000 C CNN
+F 2 "" H 5400 6050 60  0001 C CNN
+F 3 "" H 5400 6050 60  0001 C CNN
+	1    5400 6050
+	1    0    0    -1
+$EndComp
 Wire Bus Line
 	5200 5600 5200 5800
