File: hw/bus-splitter/bus-splitter.sch (KiCad schematic (older format))
At the start: 34 parts

Commit message: Feat: Initial revision of bus-splitter PCB
Parts:
- removed C? (x2): C, symbol C
- removed J? (x4): CONN_1X1, symbol CONN_1X1
- removed R? (x4): R, symbol R
- removed U?: 25LCXXX, SO8N, symbol 25LCXXX
- added C7: 100nF, Capacitors_SMD:C_0805, symbol C
- added J6: WAGO 243-723, Connector_WAGO:WAGO243, symbol CONN_1X1
- added J7: WAGO 243-724, Connector_WAGO:WAGO243, symbol CONN_1X1
- added J8: WAGO 243-721, Connector_WAGO:WAGO243, symbol CONN_1X1
- added J9: WAGO 243-722, Connector_WAGO:WAGO243, symbol CONN_1X1
- added R3: 100, Resistor:R_0805, symbol R
- C1: renamed from C?; value C -> 100µF/6V; footprint (none) -> Capacitors_SMD:C_0805
- C2, C5: renamed from C?; value C -> 100nF; footprint (none) -> Capacitors_SMD:C_0805
- C3, C4: renamed from C?; value C -> 18pF; footprint (none) -> Capacitors_SMD:C_0805
- C6: renamed from C?; value C -> 4,7nF; footprint (none) -> Capacitors_SMD:C_0805
- D1, D3: renamed from D?; footprint (none) -> Diode_SMD:D_SOT143
- D2: renamed from D?; footprint (none) -> Diode_SMD:D_SOD323
- F1: renamed from F?; footprint (none) -> Resistor:R_1206
- J1, J2, J3, J4: renamed from J?; footprint (none) -> Connector_WAGO:WAGO243
- J5: renamed from J?; footprint AVR-ISP-6 -> Connector_Header:HEADER_3x2
- R1: renamed from R?; footprint (none) -> Resistor:R_RM10.16mm
- R2: renamed from R?; value R -> 10k; footprint (none) -> Resistor:R_0805
- R4: renamed from R?; value R -> 100; footprint (none) -> Resistor:R_0805
- U1: renamed from U?; footprint AM1S-XXXX_SIL4 -> DCDC_Converter:AM1S-XXXX_SIL4
- U2, U5: renamed from U?; footprint SSOP28 -> Housings_SOIC:SO8E
- U3: renamed from U?; value CRYSTAL -> 7.3728MHz; footprint (none) -> Crystal:CRY_HC49_SMD
- U4: renamed from U?; footprint SO20L -> Housings_SOIC:SO20L
Connections:
- net labels added: /RESET, 24V_UNFUSED, A0, A1, B0, B1, RXD0, RXD1_MISO, SCK, TXD0, TXD1_MOSI, TXDEN0, TXDEN1
- wire segments 23 -> 104
- no-connect marks 2 -> 10
Other:
- moved on the sheet: C1, C2, C3, C4, C5, C6, D1, D2, D3, F1, J1, J2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

Commit message: Feat: Finished PCB for review
Parts:
- added LOGO1: OPEN_HARDWARE_1, Symbol:Symbol_OSHW-Logo_Copper, symbol OPEN_HARDWARE_1
- D2: value D -> 1N4148
- F1: value FUSE -> 0,15A
Changed lines of the file:
@@
 Sheet 1 1
 Title "bus-splitter"
-Date "2018-06-13"
+Date "2018-06-14"
 Rev "1"
 Comp "koewiba"
@@
 P 1750 2850
 F 0 "F1" H 1750 2950 50  0000 C CNN
-F 1 "FUSE" H 1750 2750 50  0000 C CNN
+F 1 "0,15A" H 1750 2750 50  0000 C CNN
 F 2 "Resistor:R_1206" H 1750 2850 60  0001 C CNN
 F 3 "" H 1750 2850 60  0000 C CNN
@@
 P 6700 4750
 F 0 "D2" H 6710 4830 50  0000 C CNN
-F 1 "D" H 6700 4675 50  0000 C CNN
+F 1 "1N4148" H 6700 4675 50  0000 C CNN
 F 2 "Diode_SMD:D_SOD323" H 6700 4750 60  0001 C CNN
 F 3 "" H 6700 4750 60  0000 C CNN
@@
 B1
 $Comp
-L GND #PWR?
+L GND #PWR022
 U 1 1 5B2108EB
 P 9800 4550
-F 0 "#PWR?" H 9800 4350 50  0001 C CNN
+F 0 "#PWR022" H 9800 4350 50  0001 C CNN
 F 1 "GND" H 9800 4440 50  0001 C CNN
 F 2 "" H 9800 4550 60  0001 C CNN
@@
 $EndComp
 Connection ~ 9800 4450
+$Comp
+L OPEN_HARDWARE_1 LOGO1
+U 1 1 5B225B1C
+P 1200 7250
+F 0 "LOGO1" H 1200 7525 50  0000 C CNN
+F 1 "OPEN_HARDWARE_1" H 1200 7025 25  0000 C CNN
+F 2 "Symbol:Symbol_OSHW-Logo_Copper" H 1200 7250 60  0001 C CNN
+F 3 "" H 1200 7250 60  0001 C CNN
+	1    1200 7250
+	1    0    0    -1
+$EndComp
 $EndSCHEMATC

Commit message: added testpoints
Parts:
- added J10: tp_vcc, Connector_Miscelleaneus:Testpoint_1mm, symbol connectors:CONN_1
- added J11: tp_gnd, Connector_Miscelleaneus:Testpoint_1mm, symbol connectors:CONN_1
- added J12: tp_txd0, Connector_Miscelleaneus:Testpoint_1mm, symbol connectors:CONN_1
- added J13: tp_rxd0, Connector_Miscelleaneus:Testpoint_1mm, symbol connectors:CONN_1
- added J14: tp_txden0, Connector_Miscelleaneus:Testpoint_1mm, symbol connectors:CONN_1
- added J15: tp_reset, Connector_Miscelleaneus:Testpoint_1mm, symbol connectors:CONN_1
- added J16: tp_txd1_mosi, Connector_Miscelleaneus:Testpoint_1mm, symbol connectors:CONN_1
- added J17: tp_rxd1_miso, Connector_Miscelleaneus:Testpoint_1mm, symbol connectors:CONN_1
- added J18: tp_sck, Connector_Miscelleaneus:Testpoint_1mm, symbol connectors:CONN_1
- added J19: tp_txden1, Connector_Miscelleaneus:Testpoint_1mm, symbol connectors:CONN_1
- C1, C2, C3, C4, C5, C6, C7: symbol C -> bus-splitter-rescue:C
- D1, D3: symbol SEMTECH_SR05 -> bus-splitter-rescue:SEMTECH_SR05
- D2: symbol D -> bus-splitter-rescue:D
- F1: symbol FUSE -> bus-splitter-rescue:FUSE
- J1, J2, J3, J4, J6, J7, J8, J9: symbol CONN_1X1 -> bus-splitter-rescue:CONN_1X1
- J5: symbol CONN-ISP-6 -> bus-splitter-rescue:CONN-ISP-6
- LOGO1: symbol OPEN_HARDWARE_1 -> bus-splitter-rescue:OPEN_HARDWARE_1
- R1: symbol Varistor -> bus-splitter-rescue:Varistor
- R2, R3, R4: symbol R -> bus-splitter-rescue:R
- U1: symbol AM1S-2405 -> bus-splitter-rescue:AM1S-2405
- U2, U5: symbol MAX487 -> bus-splitter-rescue:MAX487
- U3: symbol CRYSTAL -> bus-splitter-rescue:CRYSTAL
- U4: symbol ATTINY1634-SOIC -> bus-splitter-rescue:ATTINY1634-SOIC
Connections:
- wire segments 104 -> 140

Commit message: Added 3d images Added component placement drawings Added gerber files Fixes rescue library mess
Parts:
- C1, C2, C3, C4, C5, C6, C7: symbol bus-splitter-rescue:C -> standard:C
- D1, D3: symbol bus-splitter-rescue:SEMTECH_SR05 -> diodes:SEMTECH_SR05
- D2: symbol bus-splitter-rescue:D -> standard:D
- F1: symbol bus-splitter-rescue:FUSE -> standard:FUSE
- J1, J2, J3, J4, J6, J7, J8, J9: symbol bus-splitter-rescue:CONN_1X1 -> connectors:CONN_1X1
- J5: symbol bus-splitter-rescue:CONN-ISP-6 -> connectors:CONN-ISP-6
- LOGO1: symbol bus-splitter-rescue:OPEN_HARDWARE_1 -> logo:OPEN_HARDWARE_1
- R1: symbol bus-splitter-rescue:Varistor -> standard:Varistor
- R2, R3, R4: symbol bus-splitter-rescue:R -> standard:R
- U1: symbol bus-splitter-rescue:AM1S-2405 -> ics_regulator:AM1S-2405
- U2, U5: symbol bus-splitter-rescue:MAX487 -> ics_misc:MAX487
- U3: symbol bus-splitter-rescue:CRYSTAL -> standard:CRYSTAL
- U4: symbol bus-splitter-rescue:ATTINY1634-SOIC -> ics_controller_atmel:ATTINY1634-SOIC
Changed lines of the file:
@@
 Title "bus-splitter"
 Date "2018-09-21"
-Rev "1"
+Rev "A"
 Comp "koewiba"
 Comment1 ""
@@
 $EndDescr
 $Comp
-L bus-splitter-rescue:ATTINY1634-SOIC U4
+L ics_controller_atmel:ATTINY1634-SOIC U4
 U 1 1 5B1FC4AC
 P 6000 3800
@@
 $EndComp
 $Comp
-L bus-splitter-rescue:CRYSTAL U3
+L standard:CRYSTAL U3
 U 1 1 5B1FC51B
 P 5650 5050
@@
 $EndComp
 $Comp
-L bus-splitter-rescue:C C5
+L standard:C C5
 U 1 1 5B1FC574
 P 6200 2650
@@
 $EndComp
 $Comp
-L bus-splitter-rescue:C C4
+L standard:C C4
 U 1 1 5B1FC5E5
 P 5750 5250
@@
 $EndComp
 $Comp
-L bus-splitter-rescue:C C3
+L standard:C C3
 U 1 1 5B1FC602
 P 5200 5250
@@
 $EndComp
 $Comp
-L bus-splitter-rescue:CONN-ISP-6 J5
+L connectors:CONN-ISP-6 J5
 U 1 1 5B1FC62B
 P 8150 5150
@@
 $EndComp
 $Comp
-L bus-splitter-rescue:CONN_1X1 J1
+L connectors:CONN_1X1 J1
 U 1 1 5B1FC7EC
 P 1250 2850
@@
 $EndComp
 $Comp
-L bus-splitter-rescue:CONN_1X1 J2
+L connectors:CONN_1X1 J2
 U 1 1 5B1FC81B
 P 1250 3150
@@
 $EndComp
 $Comp
-L bus-splitter-rescue:CONN_1X1 J3
+L connectors:CONN_1X1 J3
 U 1 1 5B1FC852
 P 1250 3450
@@
 $EndComp
 $Comp
-L bus-splitter-rescue:CONN_1X1 J4
+L connectors:CONN_1X1 J4
 U 1 1 5B1FC8B1
 P 1250 3750
@@
 $EndComp
 $Comp
-L bus-splitter-rescue:FUSE F1
+L standard:FUSE F1
 U 1 1 5B1FC963
 P 1750 2850
@@
 $EndComp
 $Comp
-L bus-splitter-rescue:MAX487 U2
+L ics_misc:MAX487 U2
 U 1 1 5B1FCAC1
 P 3550 3300
@@
 $EndComp
 $Comp
-L bus-splitter-rescue:MAX487 U5
+L ics_misc:MAX487 U5
 U 1 1 5B1FCB38
 P 8850 3300
@@
 $EndComp
 $Comp
-L bus-splitter-rescue:C C2
+L standard:C C2
 U 1 1 5B1FCBA9
 P 3750 2650
@@
 $EndComp
 $Comp
-L bus-splitter-rescue:R R2
+L standard:R R2
 U 1 1 5B1FD0F2
 P 6900 4750
@@
 $EndComp
 $Comp
-L bus-splitter-rescue:C C6
+L standard:C C6
 U 1 1 5B1FD1F5
 P 6900 5250
@@
 $EndComp
 $Comp
-L bus-splitter-rescue:D D2
+L standard:D D2
 U 1 1 5B1FD25A
 P 6700 4750
@@
 $EndComp
 $Comp
-L bus-splitter-rescue:SEMTECH_SR05 D1
+L diodes:SEMTECH_SR05 D1
 U 1 1 5B1FD34A
 P 2600 4050
@@
 $EndComp
 $Comp
-L bus-splitter-rescue:SEMTECH_SR05 D3
+L diodes:SEMTECH_SR05 D3
 U 1 1 5B1FD3F5
 P 9800 4050
@@
 $EndComp
 $Comp
-L bus-splitter-rescue:Varistor R1
+L standard:Varistor R1
 U 1 1 5B1FD4A0
 P 2050 4100
@@
 $EndComp
 $Comp
-L bus-splitter-rescue:R R4
+L standard:R R4
 U 1 1 5B1FD567
 P 8050 3450
@@
 GND
 $Comp
-L bus-splitter-rescue:GND #PWR01
+L power:GND #PWR01
 U 1 1 5B1FECB7
 P 2050 4550
@@
 $EndComp
 $Comp
-L power1:+24V #PWR02
+L power:+24V #PWR02
 U 1 1 5B1FED11
 P 2050 2750
@@
 $EndComp
 $Comp
-L bus-splitter-rescue:GND #PWR03
+L power:GND #PWR03
 U 1 1 5B1FF42F
 P 3550 3950
@@
 $EndComp
 $Comp
-L bus-splitter-rescue:GND #PWR04
+L power:GND #PWR04
 U 1 1 5B1FF487
 P 3950 2750
@@
 $EndComp
 $Comp
-L power1:VCC #PWR05
+L power:VCC #PWR05
 U 1 1 5B1FF4DF
 P 3550 2550
@@
 	3550 3850 3550 3950
 $Comp
-L power1:+24V #PWR06
+L power:+24V #PWR06
 U 1 1 5B1FF8D2
 P 2050 4850
@@
 $EndComp
 $Comp
-L bus-splitter-rescue:GND #PWR07
+L power:GND #PWR07
 U 1 1 5B1FF92A
 P 2050 5450
@@
 $EndComp
 $Comp
-L bus-splitter-rescue:C C1
+L standard:C C1
 U 1 1 5B1FD7C3
 P 3350 5150
@@
 $EndComp
 $Comp
-L bus-splitter-rescue:AM1S-2405 U1
+L ics_regulator:AM1S-2405 U1
 U 1 1 5B1FC8F2
 P 2650 5150
@@
 Connection ~ 3350 5350
 $Comp
-L bus-splitter-rescue:GND #PWR08
+L power:GND #PWR08
 U 1 1 5B20E396
 P 3350 5450
@@
 Connection ~ 3350 4950
 $Comp
-L power1:VCC #PWR09
+L power:VCC #PWR09
 U 1 1 5B20E5DF
 P 3350 4850
@@
 	4800 3850 4900 3750
 $Comp
-L bus-splitter-rescue:R R3
+L standard:R R3
 U 1 1 5B20FAC2
 P 8050 3150
@@
 NoConn ~ 6700 4050
 $Comp
-L power1:VCC #PWR010
+L power:VCC #PWR010
 U 1 1 5B210DC4
 P 6000 2550
@@
 $EndComp
 $Comp
-L bus-splitter-rescue:GND #PWR011
+L power:GND #PWR011
 U 1 1 5B210E18
 P 6400 2750
@@
 	6000 4850 6000 5450
 $Comp
-L bus-splitter-rescue:GND #PWR012
+L power:GND #PWR012
 U 1 1 5B212396
 P 5200 5450
@@
 $EndComp
 $Comp
-L bus-splitter-rescue:GND #PWR013
+L power:GND #PWR013
 U 1 1 5B2123EA
 P 5750 5450
@@
 $EndComp
 $Comp
-L bus-splitter-rescue:GND #PWR014
+L power:GND #PWR014
 U 1 1 5B21243E
 P 6000 5450
@@
 $EndComp
 $Comp
-L power1:VCC #PWR015
+L power:VCC #PWR015
 U 1 1 5B2128CB
 P 8550 4950
@@
 $EndComp
 $Comp
-L bus-splitter-rescue:GND #PWR016
+L power:GND #PWR016
 U 1 1 5B21291F
 P 8550 5450
@@
 	7850 5050 7400 5050
 $Comp
-L bus-splitter-rescue:GND #PWR017
+L power:GND #PWR017
 U 1 1 5B21341E
 P 6900 5450
@@
 Connection ~ 6800 4450
 $Comp
-L power1:VCC #PWR018
+L power:VCC #PWR018
 U 1 1 5B2137A5
 P 6800 4350
@@
 	7300 3550 7400 3450
 $Comp
-L bus-splitter-rescue:C C7
+L standard:C C7
 U 1 1 5B215009
 P 9050 2650
@@
 $EndComp
 $Comp
-L power1:VCC #PWR019
+L power:VCC #PWR019
 U 1 1 5B21500F
 P 8850 2550
@@
 $EndComp
 $Comp
-L bus-splitter-rescue:GND #PWR020
+L power:GND #PWR020
 U 1 1 5B215015
 P 9250 2750
@@
 Connection ~ 8850 2650
 $Comp
-L bus-splitter-rescue:GND #PWR021
+L power:GND #PWR021
 U 1 1 5B2152E0
 P 8850 3950
@@
 	8850 3850 8850 3950
 $Comp
-L bus-splitter-rescue:CONN_1X1 J6
+L connectors:CONN_1X1 J6
 U 1 1 5B215E52
 P 10550 2850
@@
 $EndComp
 $Comp
-L bus-splitter-rescue:CONN_1X1 J7
+L connectors:CONN_1X1 J7
 U 1 1 5B215E58
 P 10550 3150
@@
 $EndComp
 $Comp
-L bus-splitter-rescue:CONN_1X1 J8
+L connectors:CONN_1X1 J8
 U 1 1 5B215E5E
 P 10550 3450
@@
 $EndComp
 $Comp
-L bus-splitter-rescue:CONN_1X1 J9
+L connectors:CONN_1X1 J9
 U 1 1 5B215E64
 P 10550 3750
@@
 B1
 $Comp
-L bus-splitter-rescue:GND #PWR022
+L power:GND #PWR022
 U 1 1 5B2108EB
 P 9800 4550
@@
 Connection ~ 9800 4450
 $Comp
-L bus-splitter-rescue:OPEN_HARDWARE_1 LOGO1
+L logo:OPEN_HARDWARE_1 LOGO1
 U 1 1 5B225B1C
 P 1200 7250
