File: hw/switch_3pole_5x/inputs.sch (KiCad schematic (older format))
At the start: 15 parts, among them J7 WAGO 233-504, J8 WAGO 233-504, J9 WAGO 233-502

Commit message: Added LED and testpoints
Parts:
- added J19: tp_button_0, Connector_Miscelleaneus:Testpoint_1mm, symbol connectors:CONN_1
- added J20: tp_button_1, Connector_Miscelleaneus:Testpoint_1mm, symbol connectors:CONN_1
- added J21: tp_button_2, Connector_Miscelleaneus:Testpoint_1mm, symbol connectors:CONN_1
- added J22: tp_button_3, Connector_Miscelleaneus:Testpoint_1mm, symbol connectors:CONN_1
- added J23: tp_button_4, Connector_Miscelleaneus:Testpoint_1mm, symbol connectors:CONN_1
- D11, D12, D13, D14, D15: symbol BAT54S -> switch_3pole_5x-rescue:BAT54S
- D21: symbol ZD -> switch_3pole_5x-rescue:ZD
- J7, J8: symbol CONN_4X1 -> switch_3pole_5x-rescue:CONN_4X1
- J9: symbol CONN_2X1 -> switch_3pole_5x-rescue:CONN_2X1
- LOGO3: symbol OPEN_HARDWARE_1 -> switch_3pole_5x-rescue:OPEN_HARDWARE_1
- R21, R22, R23, R24, R25: symbol R -> switch_3pole_5x-rescue:R
Connections:
- net button_0: now also J19.1
- net button_1: now also J20.1
- net button_2: now also J21.1
- net button_3: now also J22.1
- net button_4: now also J23.1
Changed lines of the file:
@@
-EESchema Schematic File Version 2
-LIBS:diodes
-LIBS:ics_controller_atmel
-LIBS:ics_misc
-LIBS:ics_peripheral
-LIBS:logo
-LIBS:analog_devices
-LIBS:connectors
-LIBS:display
-LIBS:encoder
-LIBS:ftdi
-LIBS:ics_40xx
-LIBS:ics_74xx
-LIBS:ics_opamp
-LIBS:ics_opto
-LIBS:ics_regulator
-LIBS:ics_signal
-LIBS:modules
-LIBS:power
-LIBS:relays
-LIBS:sensors
-LIBS:standard
-LIBS:transformer
-LIBS:transistors
+EESchema Schematic File Version 4
 LIBS:switch_3pole_5x-cache
-EELAYER 25 0
+EELAYER 26 0
 EELAYER END
 $Descr A4 11693 8268
@@
 Sheet 3 4
 Title "switch 3pole (inputs)"
-Date "2018-06-08"
+Date "2018-09-18"
 Rev "1"
 Comp "koewiba"
@@
 /button_1
 $Comp
-L +5V #PWR014
+L power1:+5V #PWR014
 U 1 1 572DD72B
 P 4250 2900
 F 0 "#PWR014" H 4250 3100 50  0001 C CNN
-F 1 "+5V" H 4250 3000 50  0000 C CNN
+F 1 "+5V" H 4250 3050 50  0000 C CNN
 F 2 "" H 4250 2900 60  0000 C CNN
 F 3 "" H 4250 2900 60  0000 C CNN
@@
 $EndComp
 $Comp
-L GND #PWR015
+L switch_3pole_5x-rescue:GND #PWR015
 U 1 1 572DD731
 P 4250 3400
@@
 $EndComp
 $Comp
-L GND #PWR016
+L switch_3pole_5x-rescue:GND #PWR016
 U 1 1 572DE6EB
 P 3925 2875
@@
 $EndComp
 $Comp
-L OPEN_HARDWARE_1 LOGO3
+L switch_3pole_5x-rescue:OPEN_HARDWARE_1 LOGO3
 U 1 1 5B10FE76
 P 975 7350
@@
 $EndComp
 $Comp
-L BAT54S D12
+L switch_3pole_5x-rescue:BAT54S D12
 U 1 1 57AB8D78
 P 4250 3150
@@
 	3925 2500 3600 2500
 Wire Wire Line
-	3925 2500 3925 2875
+	3925 2500 3925 2700
 Wire Wire Line
 	3600 2600 3850 2600
 $Comp
-L CONN_4X1 J7
+L switch_3pole_5x-rescue:CONN_4X1 J7
 U 1 1 5B0E2195
 P 3400 2550
@@
 Connection ~ 3925 2700
 $Comp
-L R R22
+L switch_3pole_5x-rescue:R R22
 U 1 1 572DD721
 P 4250 3600
@@
 $EndComp
 $Comp
-L +5V #PWR017
+L power1:+5V #PWR017
 U 1 1 5B0E2682
 P 4250 1700
 F 0 "#PWR017" H 4250 1900 50  0001 C CNN
-F 1 "+5V" H 4250 1800 50  0000 C CNN
+F 1 "+5V" H 4250 1850 50  0000 C CNN
 F 2 "" H 4250 1700 60  0000 C CNN
 F 3 "" H 4250 1700 60  0000 C CNN
@@
 $EndComp
 $Comp
-L GND #PWR018
+L switch_3pole_5x-rescue:GND #PWR018
 U 1 1 5B0E2688
 P 4250 2200
@@
 $EndComp
 $Comp
-L BAT54S D11
+L switch_3pole_5x-rescue:BAT54S D11
 U 1 1 5B0E268E
 P 4250 1950
@@
 $EndComp
 $Comp
-L R R21
+L switch_3pole_5x-rescue:R R21
 U 1 1 5B0E2694
 P 4250 2400
@@
 	4250 3350 4250 3400
 Wire Wire Line
-	5150 2400 4450 2400
-Wire Wire Line
-	4550 2400 4550 1950
+	5150 2400 4550 2400
+Wire Wire Line
+	4550 2400 4550 2200
 Wire Wire Line
 	4550 1950 4350 1950
 Wire Wire Line
-	5150 3600 4450 3600
-Wire Wire Line
-	4550 3600 4550 3150
+	5150 3600 4550 3600
+Wire Wire Line
+	4550 3600 4550 3400
 Wire Wire Line
 	4550 3150 4350 3150
@@
 /button_3
 $Comp
-L +5V #PWR019
+L power1:+5V #PWR019
 U 1 1 5B0E2FF8
 P 4250 5300
 F 0 "#PWR019" H 4250 5500 50  0001 C CNN
-F 1 "+5V" H 4250 5400 50  0000 C CNN
+F 1 "+5V" H 4250 5450 50  0000 C CNN
 F 2 "" H 4250 5300 60  0000 C CNN
 F 3 "" H 4250 5300 60  0000 C CNN
@@
 $EndComp
 $Comp
-L GND #PWR020
+L switch_3pole_5x-rescue:GND #PWR020
 U 1 1 5B0E2FFE
 P 4250 5800
@@
 $EndComp
 $Comp
-L GND #PWR021
+L switch_3pole_5x-rescue:GND #PWR021
 U 1 1 5B0E3004
 P 3925 5275
@@
 $EndComp
 $Comp
-L BAT54S D14
+L switch_3pole_5x-rescue:BAT54S D14
 U 1 1 5B0E300A
 P 4250 5550
@@
 	3925 4900 3600 4900
 Wire Wire Line
-	3925 4900 3925 5275
+	3925 4900 3925 5100
 Wire Wire Line
 	3600 5000 3850 5000
 $Comp
-L CONN_4X1 J8
+L switch_3pole_5x-rescue:CONN_4X1 J8
 U 1 1 5B0E3013
 P 3400 4950
@@
 Connection ~ 3925 5100
 $Comp
-L R R24
+L switch_3pole_5x-rescue:R R24
 U 1 1 5B0E301B
 P 4250 6000
@@
 $EndComp
 $Comp
-L +5V #PWR022
+L power1:+5V #PWR022
 U 1 1 5B0E3021
 P 4250 4100
 F 0 "#PWR022" H 4250 4300 50  0001 C CNN
-F 1 "+5V" H 4250 4200 50  0000 C CNN
+F 1 "+5V" H 4250 4250 50  0000 C CNN
 F 2 "" H 4250 4100 60  0000 C CNN
 F 3 "" H 4250 4100 60  0000 C CNN
@@
 $EndComp
 $Comp
-L GND #PWR023
+L switch_3pole_5x-rescue:GND #PWR023
 U 1 1 5B0E3027
 P 4250 4600
@@
 $EndComp
 $Comp
-L BAT54S D13
+L switch_3pole_5x-rescue:BAT54S D13
 U 1 1 5B0E302D
 P 4250 4350
@@
 $EndComp
 $Comp
-L R R23
+L switch_3pole_5x-rescue:R R23
 U 1 1 5B0E3033
 P 4250 4800
@@
 	4250 5750 4250 5800
 Wire Wire Line
-	5150 4800 4450 4800
-Wire Wire Line
-	4550 4800 4550 4350
+	5150 4800 4550 4800
+Wire Wire Line
+	4550 4800 4550 4600
 Wire Wire Line
 	4550 4350 4350 4350
 Wire Wire Line
-	5150 6000 4450 6000
-Wire Wire Line
-	4550 6000 4550 5550
+	5150 6000 4550 6000
+Wire Wire Line
+	4550 6000 4550 5800
 Wire Wire Line
 	4550 5550 4350 5550
@@
 /button_4
 $Comp
-L +5V #PWR024
+L power1:+5V #PWR024
 U 1 1 5B0E32D9
 P 7350 1700
 F 0 "#PWR024" H 7350 1900 50  0001 C CNN
-F 1 "+5V" H 7350 1800 50  0000 C CNN
+F 1 "+5V" H 7350 1850 50  0000 C CNN
 F 2 "" H 7350 1700 60  0000 C CNN
 F 3 "" H 7350 1700 60  0000 C CNN
@@
 $EndComp
 $Comp
-L GND #PWR025
+L switch_3pole_5x-rescue:GND #PWR025
 U 1 1 5B0E32DF
 P 7350 2200
@@
 $EndComp
 $Comp
-L BAT54S D15
+L switch_3pole_5x-rescue:BAT54S D15
 U 1 1 5B0E32E5
 P 7350 1950
@@
 $EndComp
 $Comp
-L R R25
+L switch_3pole_5x-rescue:R R25
 U 1 1 5B0E32EB
 P 7350 2400
@@
 	7150 2400 6700 2400
 Wire Wire Line
-	8250 2400 7550 2400
-Wire Wire Line
-	7650 2400 7650 1950
+	8250 2400 7650 2400
+Wire Wire Line
+	7650 2400 7650 2200
 Wire Wire Line
 	7650 1950 7450 1950
@@
 button_4
 $Comp
-L ZD D21
+L switch_3pole_5x-rescue:ZD D21
 U 1 1 5B0E3DD6
 P 7550 4800
@@
 $EndComp
 $Comp
-L +5V #PWR026
+L power1:+5V #PWR026
 U 1 1 5B0E3F0E
 P 7550 4500
 F 0 "#PWR026" H 7550 4700 50  0001 C CNN
-F 1 "+5V" H 7550 4610 50  0000 C CNN
+F 1 "+5V" H 7550 4650 50  0000 C CNN
 F 2 "" H 7550 4500 60  0001 C CNN
 F 3 "" H 7550 4500 60  0001 C CNN
@@
 $EndComp
 $Comp
-L GND #PWR027
+L switch_3pole_5x-rescue:GND #PWR027
 U 1 1 5B0E3FFA
 P 7550 5100
@@
 Place close to inputs!
 $Comp
-L CONN_2X1 J9
+L switch_3pole_5x-rescue:CONN_2X1 J9
 U 1 1 5B1A4C2C
 P 6500 2450
@@
 $EndComp
 $Comp
-L GND #PWR028
+L switch_3pole_5x-rescue:GND #PWR028
 U 1 1 5B0E32BC
 P 6800 2600
@@
 Wire Wire Line
 	6800 2500 6800 2600
+Wire Wire Line
+	3925 2700 3925 2875
+Wire Wire Line
+	4550 2400 4450 2400
+Wire Wire Line
+	4550 3600 4450 3600
+Wire Wire Line
+	3925 5100 3925 5275
+Wire Wire Line
+	4550 4800 4450 4800
+Wire Wire Line
+	4550 6000 4450 6000
+Wire Wire Line
+	7650 2400 7550 2400
+$Comp
+L connectors:CONN_1 J19
+U 1 1 5BA165F9
+P 4750 2200
+F 0 "J19" H 4791 2236 50  0000 L CNN
+F 1 "tp_button_0" H 4791 2164 25  0000 L CNN
+F 2 "Connector_Miscelleaneus:Testpoint_1mm" H 4750 2200 60  0001 C CNN
+F 3 "" H 4750 2200 60  0000 C CNN
+	1    4750 2200
+	1    0    0    -1
+$EndComp
+$Comp
+L connectors:CONN_1 J20
+U 1 1 5BA166D5
+P 4750 3400
+F 0 "J20" H 4791 3436 50  0000 L CNN
+F 1 "tp_button_1" H 4791 3364 25  0000 L CNN
+F 2 "Connector_Miscelleaneus:Testpoint_1mm" H 4750 3400 60  0001 C CNN
+F 3 "" H 4750 3400 60  0000 C CNN
+	1    4750 3400
+	1    0    0    -1
+$EndComp
+$Comp
+L connectors:CONN_1 J21
+U 1 1 5BA16774
+P 4750 4600
+F 0 "J21" H 4791 4636 50  0000 L CNN
+F 1 "tp_button_2" H 4791 4564 25  0000 L CNN
+F 2 "Connector_Miscelleaneus:Testpoint_1mm" H 4750 4600 60  0001 C CNN
+F 3 "" H 4750 4600 60  0000 C CNN
+	1    4750 4600
+	1    0    0    -1
+$EndComp
+$Comp
+L connectors:CONN_1 J22
+U 1 1 5BA167E4
+P 4750 5800
+F 0 "J22" H 4791 5836 50  0000 L CNN
+F 1 "tp_button_3" H 4791 5764 25  0000 L CNN
+F 2 "Connector_Miscelleaneus:Testpoint_1mm" H 4750 5800 60  0001 C CNN
+F 3 "" H 4750 5800 60  0000 C CNN
+	1    4750 5800
+	1    0    0    -1
+$EndComp
+$Comp
+L connectors:CONN_1 J23
+U 1 1 5BA16905
+P 7850 2200
+F 0 "J23" H 7891 2236 50  0000 L CNN
+F 1 "tp_button_4" H 7891 2164 25  0000 L CNN
+F 2 "Connector_Miscelleaneus:Testpoint_1mm" H 7850 2200 60  0001 C CNN
+F 3 "" H 7850 2200 60  0000 C CNN
+	1    7850 2200
+	1    0    0    -1
+$EndComp
+Wire Wire Line
+	4650 2200 4550 2200
+Connection ~ 4550 2200
+Wire Wire Line
+	4550 2200 4550 1950
+Wire Wire Line
+	4650 3400 4550 3400
+Connection ~ 4550 3400
+Wire Wire Line
+	4550 3400 4550 3150
+Wire Wire Line
+	7750 2200 7650 2200
+Connection ~ 7650 2200
+Wire Wire Line
+	7650 2200 7650 1950
+Wire Wire Line
+	4650 4600 4550 4600
+Connection ~ 4550 4600
+Wire Wire Line
+	4550 4600 4550 4350
+Wire Wire Line
+	4650 5800 4550 5800
+Connection ~ 4550 5800
+Wire Wire Line
+	4550 5800 4550 5550
 $EndSCHEMATC

Commit message: fixed switch_3pole_5x library references added component placement drawings updated 3d images and gerber files
Parts:
- D11, D12, D13, D14, D15: symbol switch_3pole_5x-rescue:BAT54S -> diodes:BAT54S
- D21: symbol switch_3pole_5x-rescue:ZD -> standard:ZD
- J7, J8: symbol switch_3pole_5x-rescue:CONN_4X1 -> connectors:CONN_4X1
- J9: symbol switch_3pole_5x-rescue:CONN_2X1 -> connectors:CONN_2X1
- LOGO3: symbol switch_3pole_5x-rescue:OPEN_HARDWARE_1 -> logo:OPEN_HARDWARE_1
- R21, R22, R23, R24, R25: symbol switch_3pole_5x-rescue:R -> standard:R
Changed lines of the file:
@@
 Title "switch 3pole (inputs)"
 Date "2018-09-18"
-Rev "1"
+Rev "A"
 Comp "koewiba"
 Comment1 ""
@@
 /button_1
 $Comp
-L power1:+5V #PWR014
+L power:+5V #PWR014
 U 1 1 572DD72B
 P 4250 2900
@@
 $EndComp
 $Comp
-L switch_3pole_5x-rescue:GND #PWR015
+L power:GND #PWR015
 U 1 1 572DD731
 P 4250 3400
@@
 $EndComp
 $Comp
-L switch_3pole_5x-rescue:GND #PWR016
+L power:GND #PWR016
 U 1 1 572DE6EB
 P 3925 2875
@@
 $EndComp
 $Comp
-L switch_3pole_5x-rescue:OPEN_HARDWARE_1 LOGO3
+L logo:OPEN_HARDWARE_1 LOGO3
 U 1 1 5B10FE76
 P 975 7350
@@
 $EndComp
 $Comp
-L switch_3pole_5x-rescue:BAT54S D12
+L diodes:BAT54S D12
 U 1 1 57AB8D78
 P 4250 3150
@@
 	3600 2600 3850 2600
 $Comp
-L switch_3pole_5x-rescue:CONN_4X1 J7
+L connectors:CONN_4X1 J7
 U 1 1 5B0E2195
 P 3400 2550
@@
 Connection ~ 3925 2700
 $Comp
-L switch_3pole_5x-rescue:R R22
+L standard:R R22
 U 1 1 572DD721
 P 4250 3600
@@
 $EndComp
 $Comp
-L power1:+5V #PWR017
+L power:+5V #PWR017
 U 1 1 5B0E2682
 P 4250 1700
@@
 $EndComp
 $Comp
-L switch_3pole_5x-rescue:GND #PWR018
+L power:GND #PWR018
 U 1 1 5B0E2688
 P 4250 2200
@@
 $EndComp
 $Comp
-L switch_3pole_5x-rescue:BAT54S D11
+L diodes:BAT54S D11
 U 1 1 5B0E268E
 P 4250 1950
@@
 $EndComp
 $Comp
-L switch_3pole_5x-rescue:R R21
+L standard:R R21
 U 1 1 5B0E2694
 P 4250 2400
@@
 /button_3
 $Comp
-L power1:+5V #PWR019
+L power:+5V #PWR019
 U 1 1 5B0E2FF8
 P 4250 5300
@@
 $EndComp
 $Comp
-L switch_3pole_5x-rescue:GND #PWR020
+L power:GND #PWR020
 U 1 1 5B0E2FFE
 P 4250 5800
@@
 $EndComp
 $Comp
-L switch_3pole_5x-rescue:GND #PWR021
+L power:GND #PWR021
 U 1 1 5B0E3004
 P 3925 5275
@@
 $EndComp
 $Comp
-L switch_3pole_5x-rescue:BAT54S D14
+L diodes:BAT54S D14
 U 1 1 5B0E300A
 P 4250 5550
@@
 	3600 5000 3850 5000
 $Comp
-L switch_3pole_5x-rescue:CONN_4X1 J8
+L connectors:CONN_4X1 J8
 U 1 1 5B0E3013
 P 3400 4950
@@
 Connection ~ 3925 5100
 $Comp
-L switch_3pole_5x-rescue:R R24
+L standard:R R24
 U 1 1 5B0E301B
 P 4250 6000
@@
 $EndComp
 $Comp
-L power1:+5V #PWR022
+L power:+5V #PWR022
 U 1 1 5B0E3021
 P 4250 4100
@@
 $EndComp
 $Comp
-L switch_3pole_5x-rescue:GND #PWR023
+L power:GND #PWR023
 U 1 1 5B0E3027
 P 4250 4600
@@
 $EndComp
 $Comp
-L switch_3pole_5x-rescue:BAT54S D13
+L diodes:BAT54S D13
 U 1 1 5B0E302D
 P 4250 4350
@@
 $EndComp
 $Comp
-L switch_3pole_5x-rescue:R R23
+L standard:R R23
 U 1 1 5B0E3033
 P 4250 4800
@@
 /button_4
 $Comp
-L power1:+5V #PWR024
+L power:+5V #PWR024
 U 1 1 5B0E32D9
 P 7350 1700
@@
 $EndComp
 $Comp
-L switch_3pole_5x-rescue:GND #PWR025
+L power:GND #PWR025
 U 1 1 5B0E32DF
 P 7350 2200
@@
 $EndComp
 $Comp
-L switch_3pole_5x-rescue:BAT54S D15
+L diodes:BAT54S D15
 U 1 1 5B0E32E5
 P 7350 1950
@@
 $EndComp
 $Comp
-L switch_3pole_5x-rescue:R R25
+L standard:R R25
 U 1 1 5B0E32EB
 P 7350 2400
@@
 button_4
 $Comp
-L switch_3pole_5x-rescue:ZD D21
+L standard:ZD D21
 U 1 1 5B0E3DD6
 P 7550 4800
@@
 $EndComp
 $Comp
-L power1:+5V #PWR026
+L power:+5V #PWR026
 U 1 1 5B0E3F0E
 P 7550 4500
@@
 $EndComp
 $Comp
-L switch_3pole_5x-rescue:GND #PWR027
+L power:GND #PWR027
 U 1 1 5B0E3FFA
 P 7550 5100
@@
 Place close to inputs!
 $Comp
-L switch_3pole_5x-rescue:CONN_2X1 J9
+L connectors:CONN_2X1 J9
 U 1 1 5B1A4C2C
 P 6500 2450
@@
 $EndComp
 $Comp
-L switch_3pole_5x-rescue:GND #PWR028
+L power:GND #PWR028
 U 1 1 5B0E32BC
 P 6800 2600
