File: hw/switch_3pole_5x/switch_3pole_5x.sch (KiCad schematic (older format))
At the start: 1 part

Commit message: Added LED and testpoints
Parts:
- LOGO1: symbol OPEN_HARDWARE_1 -> switch_3pole_5x-rescue:OPEN_HARDWARE_1
Changed lines of the file:
@@
-EESchema Schematic File Version 2
-LIBS:diodes
-LIBS:ics_controller_atmel
-LIBS:ics_misc
-LIBS:ics_peripheral
-LIBS:logo
-LIBS:analog_devices
-LIBS:connectors
-LIBS:display
-LIBS:encoder
-LIBS:ftdi
-LIBS:ics_40xx
-LIBS:ics_74xx
-LIBS:ics_opamp
-LIBS:ics_opto
-LIBS:ics_regulator
-LIBS:ics_signal
-LIBS:modules
-LIBS:power
-LIBS:relays
-LIBS:sensors
-LIBS:standard
-LIBS:transformer
-LIBS:transistors
+EESchema Schematic File Version 4
 LIBS:switch_3pole_5x-cache
-EELAYER 25 0
+EELAYER 26 0
 EELAYER END
 $Descr A4 11693 8268
@@
 Sheet 1 4
 Title "switch 3pole 5x"
-Date "2018-06-08"
+Date "2018-09-18"
 Rev "1"
 Comp "koewiba"
@@
 $EndDescr
 $Comp
-L +5V #PWR01
+L power1:+5V #PWR01
 U 1 1 572DAEDB
 P 6450 3350
 F 0 "#PWR01" H 6450 3550 50  0001 C CNN
-F 1 "+5V" H 6450 3460 50  0000 C CNN
+F 1 "+5V" H 6450 3500 50  0000 C CNN
 F 2 "" H 6450 3350 60  0000 C CNN
 F 3 "" H 6450 3350 60  0000 C CNN
@@
 $EndComp
 $Comp
-L +24V #PWR02
+L power1:+24V #PWR02
 U 1 1 572DAF09
 P 4750 3350
 F 0 "#PWR02" H 4750 3550 50  0001 C CNN
-F 1 "+24V" H 4750 3460 50  0000 C CNN
+F 1 "+24V" H 4750 3500 50  0000 C CNN
 F 2 "" H 4750 3350 60  0000 C CNN
 F 3 "" H 4750 3350 60  0000 C CNN
@@
 $EndComp
 $Comp
-L OPEN_HARDWARE_1 LOGO1
+L switch_3pole_5x-rescue:OPEN_HARDWARE_1 LOGO1
 U 1 1 572E288C
 P 1025 7400
@@
 $EndSheet
 $Comp
-L GND #PWR03
+L switch_3pole_5x-rescue:GND #PWR03
 U 1 1 578B8717
 P 6450 4900
@@
 Wire Wire Line
 	7600 3450 7150 3450
-Wire Bus Line
-	7050 3550 7050 5150
 Text Label 3750 3450 0    40   ~ 0
 /button_0
@@
 	4750 4100 5250 4100
 Wire Bus Line
-	6800 5050 6800 3700
-Wire Bus Line
-	4350 3550 4350 5050
-Wire Bus Line
 	4350 5050 6800 5050
 Text Label 5100 5150 0    40   ~ 0
@@
 relay_4
 Wire Bus Line
-	4650 3900 4650 5150
-Wire Bus Line
 	4650 5150 7050 5150
 Text Label 7150 3600 0    40   ~ 0
@@
 Wire Wire Line
 	7150 4050 7600 4050
+Wire Bus Line
+	7050 3550 7050 5150
+Wire Bus Line
+	4350 3550 4350 5050
+Wire Bus Line
+	4650 3900 4650 5150
+Wire Bus Line
+	6800 3700 6800 5050
 $EndSCHEMATC

Commit message: fixed switch_3pole_5x library references added component placement drawings updated 3d images and gerber files
Parts:
- LOGO1: symbol switch_3pole_5x-rescue:OPEN_HARDWARE_1 -> logo:OPEN_HARDWARE_1
Changed lines of the file:
@@
 Title "switch 3pole 5x"
 Date "2018-09-18"
-Rev "1"
+Rev "A"
 Comp "koewiba"
 Comment1 ""
@@
 $EndDescr
 $Comp
-L power1:+5V #PWR01
+L power:+5V #PWR01
 U 1 1 572DAEDB
 P 6450 3350
@@
 $EndComp
 $Comp
-L power1:+24V #PWR02
+L power:+24V #PWR02
 U 1 1 572DAF09
 P 4750 3350
@@
 $EndComp
 $Comp
-L switch_3pole_5x-rescue:OPEN_HARDWARE_1 LOGO1
+L logo:OPEN_HARDWARE_1 LOGO1
 U 1 1 572E288C
 P 1025 7400
@@
 $EndSheet
 $Comp
-L switch_3pole_5x-rescue:GND #PWR03
+L power:GND #PWR03
 U 1 1 578B8717
 P 6450 4900
